File: jared_tv_remote/3 - complex pcb.kicad_pcb (KiCad board)
At the start: 2 copper layers, 45 x 100 mm, 48 parts, among them J1 Solar_Panel, J2 USB_C_Receptacle_USB2.0_14P, J3 Solar_Panel_Back, Q1 Q_NPN, SW1 Power, SW10 Back, SW11 Home, SW12 Source, SW13 C1, SW14 C2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

Commit message: updates
Parts:
- SW1, SW10, SW11, SW12, SW13, SW14, SW15, SW2, SW3, SW4, SW5, SW6, SW7, SW8, SW9: footprint Button_Switch_SMD:SW_SPST_CK_RS282G05A3 -> Button_Switch_SMD:SW_SPST_B3U-1000P
- moved C4 134.9 mm to (164.9, 141.2)
- moved D5 134.9 mm to (163.3, 53.9)
- moved C1 134.9 mm to (138.5, 140.7)
- moved C10 134.9 mm to (151.0, 116.4)
- moved C11 134.9 mm to (149.0, 116.4)
- moved C2 134.9 mm to (146.5, 131.4)
- moved C3 134.9 mm to (159.7, 139.5)
- moved C5 134.9 mm to (159.7, 145.2)
- moved C6 134.9 mm to (142.0, 124.4)
- moved C7 134.9 mm to (142.0, 126.4)
- moved C8 134.9 mm to (147.0, 116.4)
- moved C9 134.9 mm to (157.0, 119.9)
- moved D1 134.9 mm to (159.0, 144.2)
- moved D2 134.9 mm to (148.5, 51.7)
- moved D3 134.9 mm to (133.5, 54.0)
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Routing:
- net /ROW2: track 48.9 -> 43.7 mm
- net /IR_RX: track 32.0 -> 37.0 mm
- net /ROW3: track 34.5 -> 39.0 mm
- net /ROW4: track 48.4 -> 51.9 mm
- net GND: track 2.34 -> 5.48 mm, vias 3 -> 9
- net /COL2: track 79.8 -> 76.8 mm
- net /COL1: track 64.8 -> 67.2 mm
- net /VBUS: track 31.9 -> 34.2 mm
- net /COL0: track 52.2 -> 54.3 mm
- net /ROW1: track 50.6 -> 52.6 mm
- net +3V3: track 151.3 -> 152.8 mm
- net /IR_TX: track 87.1 -> 88.2 mm
- net /USB_DP: track 23.5 -> 22.8 mm
- net /ROW0: track 82.5 -> 83.2 mm
- net /Power Supply/VSTOR: track 134.1 -> 133.6 mm
