File: jared_tv_remote/peripherals.kicad_sch (KiCad schematic)
At the start: 24 parts, among them Q1 Q_NPN, SW1 Power, SW10 Back, SW11 Home, SW12 Source, SW13 C1, SW14 C2, SW15 Learn, SW2 Up, SW3 Mute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

Commit message: updates
Parts:
- removed D2: IR_940nm, LED_THT:LED_D5.0mm, symbol Device:LED
- added U4: E6QYDD1204-IRA940NM, E6QYDD1204-IRA940nm:LED-SMD_L3.2-W2.1-R-FD, symbol E6QYDD1204-IRA940nm:E6QYDD1204-IRA940NM
- SW1, SW10, SW11, SW12, SW13, SW14, SW15, SW2, SW3, SW4, SW5, SW6, SW7, SW8, SW9: footprint Button_Switch_SMD:SW_SPST_CK_RS282G05A3 -> Button_Switch_SMD:SW_SPST_B3U-1000P
Connections:
- net +3V3: now also U4.1 (-)
- net at R5.2: now also U4.2 (+)
Changed lines of the file:
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@@
 	(wire
 		(pts
-			(xy 73.66 22.86) (xy 73.66 26.67)
+			(xy 50.8 93.98) (xy 49.53 93.98)
 		)
 		(stroke
@@
 	(wire
 		(pts
-			(xy 50.8 93.98) (xy 49.53 93.98)
+			(xy 58.42 93.98) (xy 62.23 93.98)
 		)
 		(stroke
@@
 	(wire
 		(pts
-			(xy 58.42 93.98) (xy 62.23 93.98)
+			(xy 64.77 53.34) (xy 66.04 53.34)
 		)
 		(stroke
@@
 	(wire
 		(pts
-			(xy 64.77 53.34) (xy 66.04 53.34)
+			(xy 73.66 58.42) (xy 73.66 59.69)
 		)
 		(stroke
@@
 	(wire
 		(pts
-			(xy 73.66 58.42) (xy 73.66 59.69)
+			(xy 71.12 93.98) (xy 72.39 93.98)
 		)
 		(stroke
@@
 	(wire
 		(pts
-			(xy 71.12 93.98) (xy 72.39 93.98)
+			(xy 82.55 132.08) (xy 86.36 132.08)
 		)
 		(stroke
@@
 	(wire
 		(pts
-			(xy 82.55 132.08) (xy 86.36 132.08)
+			(xy 86.36 132.08) (xy 86.36 137.16)
 		)
 		(stroke
@@
 	(wire
 		(pts
-			(xy 86.36 132.08) (xy 86.36 137.16)
+			(xy 62.23 90.17) (xy 62.23 93.98)
 		)
 		(stroke
@@
 	(wire
 		(pts
-			(xy 62.23 90.17) (xy 62.23 93.98)
+			(xy 73.66 48.26) (xy 73.66 46.99)
 		)
 		(stroke
@@
 	(wire
 		(pts
-			(xy 73.66 48.26) (xy 73.66 46.99)
+			(xy 73.66 39.37) (xy 73.66 34.29)
 		)
 		(stroke
@@
 	(wire
 		(pts
-			(xy 73.66 39.37) (xy 73.66 34.29)
+			(xy 62.23 93.98) (xy 63.5 93.98)
 		)
 		(stroke
@@
 		)
 	)
-	(wire
-		(pts
-			(xy 62.23 93.98) (xy 63.5 93.98)
-		)
-		(stroke
-			(width 0)
-			(type default)
-		)
-	)
 	(label "ROW2"
 		(at 201.93 90.17 180)
@@
 			)
 		)
-		(property "Footprint" "Button_Switch_SMD:SW_SPST_CK_RS282G05A3"
+		(property "Footprint" "Button_Switch_SMD:SW_SPST_B3U-1000P"
 			(at 172.72 92.71 0)
 			(hide yes)
@@
 			)
 		)
-		(property "Footprint" "Button_Switch_SMD:SW_SPST_CK_RS282G05A3"
+		(property "Footprint" "Button_Switch_SMD:SW_SPST_B3U-1000P"
 			(at 207.01 77.47 0)
 			(hide yes)
@@
 			)
 		)
-		(property "Footprint" "Button_Switch_SMD:SW_SPST_CK_RS282G05A3"
+		(property "Footprint" "Button_Switch_SMD:SW_SPST_B3U-1000P"
 			(at 207.01 100.33 0)
 			(hide yes)
@@
 			)
 		)
-		(property "Footprint" "Button_Switch_SMD:SW_SPST_CK_RS282G05A3"
+		(property "Footprint" "Button_Switch_SMD:SW_SPST_B3U-1000P"
 			(at 138.43 85.09 0)
 			(hide yes)
@@
 			)
 		)
-		(property "Footprint" "Button_Switch_SMD:SW_SPST_CK_RS282G05A3"
+		(property "Footprint" "Button_Switch_SMD:SW_SPST_B3U-1000P"
 			(at 207.01 85.09 0)
 			(hide yes)
@@
 	(symbol
 		(lib_id "power:+3V3")
-		(at 73.66 22.86 0)
+		(at 73.66 24.13 0)
 		(unit 1)
 		(body_style 1)
@@
 		(dnp no)
 		(property "Reference" "#PWR4"
-			(at 73.66 26.67 0)
+			(at 73.66 27.94 0)
 			(hide yes)
 			(show_name no)
@@
 		)
 		(property "Value" "+3V3"
-			(at 73.66 19.304 0)
+			(at 73.66 20.574 0)
 			(show_name no)
 			(do_not_autoplace no)
@@
 		)
 		(property "Footprint" ""
-			(at 73.66 22.86 0)
+			(at 73.66 24.13 0)
 			(hide yes)
 			(show_name no)
@@
 		)
 		(property "Datasheet" ""
-			(at 73.66 22.86 0)
+			(at 73.66 24.13 0)
 			(hide yes)
 			(show_name no)
@@
 		)
 		(property "Description" "Power symbol creates a global label with name \"+3V3\""
-			(at 73.66 22.86 0)
+			(at 73.66 24.13 0)
 			(hide yes)
 			(show_name no)
@@
 			)
 		)
-		(property "Footprint" "Button_Switch_SMD:SW_SPST_CK_RS282G05A3"
+		(property "Footprint" "Button_Switch_SMD:SW_SPST_B3U-1000P"
 			(at 172.72 85.09 0)
 			(hide yes)
@@
 			)
 		)
-		(property "Footprint" "Button_Switch_SMD:SW_SPST_CK_RS282G05A3"
+		(property "Footprint" "Button_Switch_SMD:SW_SPST_B3U-1000P"
 			(at 138.43 100.33 0)
 			(hide yes)
@@
 			)
 		)
-		(property "Footprint" "Button_Switch_SMD:SW_SPST_CK_RS282G05A3"
+		(property "Footprint" "Button_Switch_SMD:SW_SPST_B3U-1000P"
 			(at 172.72 100.33 0)
 			(hide yes)
@@
 			)
 		)
-		(property "Footprint" "Button_Switch_SMD:SW_SPST_CK_RS282G05A3"
+		(property "Footprint" "Button_Switch_SMD:SW_SPST_B3U-1000P"
 			(at 138.43 69.85 0)
 			(hide yes)
@@
 			)
 		)
-		(property "Footprint" "Button_Switch_SMD:SW_SPST_CK_RS282G05A3"
+		(property "Footprint" "Button_Switch_SMD:SW_SPST_B3U-1000P"
 			(at 207.01 69.85 0)
 			(hide yes)
@@
 			)
 		)
-		(property "Footprint" "Button_Switch_SMD:SW_SPST_CK_RS282G05A3"
+		(property "Footprint" "Button_Switch_SMD:SW_SPST_B3U-1000P"
 			(at 172.72 69.85 0)
 			(hide yes)
@@
 			)
 		)
-		(property "Footprint" "Button_Switch_SMD:SW_SPST_CK_RS282G05A3"
+		(property "Footprint" "Button_Switch_SMD:SW_SPST_B3U-1000P"
 			(at 207.01 92.71 0)
 			(hide yes)
@@
 	)
 	(symbol
+		(lib_id "E6QYDD1204-IRA940nm:E6QYDD1204-IRA940NM")
+		(at 73.66 29.21 90)
+		(unit 1)
+		(body_style 1)
+		(exclude_from_sim no)
+		(in_bom yes)
+		(on_board yes)
+		(in_pos_files yes)
+		(dnp no)
+		(fields_autoplaced yes)
+		(property "Reference" "U4"
+			(at 77.47 26.6699 90)
+			(show_name no)
+			(do_not_autoplace no)
+			(effects
+				(font
+					(size 1.27 1.27)
+				)
+				(justify right)
+			)
+		)
+		(property "Value" "E6QYDD1204-IRA940NM"
+			(at 77.47 29.2099 90)
+			(show_name no)
+			(do_not_autoplace no)
+			(effects
+				(font
+					(size 1.27 1.27)
+				)
+				(justify right)
+			)
+		)
+		(property "Footprint" "E6QYDD1204-IRA940nm:LED-SMD_L3.2-W2.1-R-FD"
+			(at 81.28 29.21 0)
+			(hide yes)
+			(show_name no)
+			(do_not_autoplace no)
+			(effects
+				(font
+					(size 1.27 1.27)
+				)
+			)
+		)
+		(property "Datasheet" "https://lcsc.com/product-detail/New-Arrivals_EKINGLUX-E6QYDD1204-IRA940nm_C396649.html"
+			(at 83.82 29.21 0)
+			(hide yes)
+			(show_name no)
+			(do_not_autoplace no)
+			(effects
+				(font
+					(size 1.27 1.27)
+				)
+			)
+		)
+		(property "Description" ""
+			(at 73.66 29.21 0)
+			(hide yes)
+			(show_name no)
+			(do_not_autoplace no)
+			(effects
+				(font
+					(size 1.27 1.27)
+				)
+			)
+		)
+		(property "LCSC Part" "C396649"
+			(at 86.36 29.21 0)
+			(hide yes)
+			(show_name no)
+			(do_not_autoplace no)
+			(effects
+				(font
+					(size 1.27 1.27)
+				)
+			)
+		)
+		(pin "2"
+		)
+		(pin "1"
+		)
+		(instances
+			(project ""
+				(path "/9fdc1b44-fae0-464f-8449-2cd33e53f6ad/059ebac3-52af-4ed5-bc20-6bf6d2796db6"
+					(reference "U4")
+					(unit 1)
+				)
+			)
+		)
+	)
+	(symbol
 		(lib_id "power:+3V3")
 		(at 62.23 90.17 0)
@@
 			)
 		)
-		(property "Footprint" "Button_Switch_SMD:SW_SPST_CK_RS282G05A3"
+		(property "Footprint" "Button_Switch_SMD:SW_SPST_B3U-1000P"
 			(at 138.43 92.71 0)
 			(hide yes)
@@
 			)
 		)
-		(property "Footprint" "Button_Switch_SMD:SW_SPST_CK_RS282G05A3"
+		(property "Footprint" "Button_Switch_SMD:SW_SPST_B3U-1000P"
 			(at 172.72 77.47 0)
 			(hide yes)
@@
 			)
 		)
-		(property "Footprint" "Button_Switch_SMD:SW_SPST_CK_RS282G05A3"
+		(property "Footprint" "Button_Switch_SMD:SW_SPST_B3U-1000P"
 			(at 138.43 77.47 0)
 			(hide yes)
@@
 					(unit 1)
 				)
-			)
-		)
-	)
-	(symbol
-		(lib_id "Device:LED")
-		(at 73.66 30.48 270)
-		(unit 1)
-		(body_style 1)
-		(exclude_from_sim no)
-		(in_bom yes)
-		(on_board yes)
-		(in_pos_files yes)
-		(dnp no)
-		(property "Reference" "D2"
-			(at 76.2 30.48 0)
-			(show_name no)
-			(do_not_autoplace no)
-			(effects
-				(font
-					(size 1.27 1.27)
-				)
-			)
-		)
-		(property "Value" "IR_940nm"
-			(at 71.12 30.48 0)
-			(show_name no)
-			(do_not_autoplace no)
-			(effects
-				(font
-					(size 1.27 1.27)
-				)
-			)
-		)
-		(property "Footprint" "LED_THT:LED_D5.0mm"
-			(at 73.66 30.48 0)
-			(hide yes)
-			(show_name no)
-			(do_not_autoplace no)
-			(effects
-				(font
-					(size 1.27 1.27)
-				)
-			)
-		)
-		(property "Datasheet" ""
-			(at 73.66 30.48 0)
-			(hide yes)
-			(show_name no)
-			(do_not_autoplace no)
-			(effects
-				(font
-					(size 1.27 1.27)
-				)
-			)
-		)
-		(property "Description" "Light emitting diode"
-			(at 73.66 30.48 0)
-			(hide yes)
-			(show_name no)
-			(do_not_autoplace no)
-			(effects
-				(font
-					(size 1.27 1.27)
-				)
-			)
-		)
-		(property "Sim.Pins" "1=K 2=A"
-			(at 73.66 30.48 0)
-			(hide yes)
-			(show_name no)
-			(do_not_autoplace no)
-			(effects
-				(font
-					(size 1.27 1.27)
-				)
-			)
-		)
-		(pin "1"
-		)
-		(pin "2"
-		)
-		(instances
-			(project ""
-				(path "/9fdc1b44-fae0-464f-8449-2cd33e53f6ad/059ebac3-52af-4ed5-bc20-6bf6d2796db6"
-					(reference "D2")
-					(unit 1)
-				)

Commit message: new boards
Parts:
- SW1, SW10, SW11, SW12, SW13, SW14, SW15, SW2, SW3, SW4, SW5, SW6, SW7, SW8, SW9: footprint Button_Switch_SMD:SW_SPST_B3U-1000P -> Button_Switch_SMD:SW_SPST_B3SL-1002P
Other:
- moved on the sheet: C1, D1, Q1, R1, R3, R4, R5, U1, U4
