File: jared_tv_remote/remote.kicad_pcb (KiCad board)
At the start: 2 copper layers, 45 x 100 mm, 48 parts, among them J1 Solar_Panel, J2 USB_C_Receptacle_USB2.0_14P, J3 Solar_Panel_Back, Q1 Q_NPN, SW1 Power, SW10 Back, SW11 Home, SW12 Source, SW13 C1, SW14 C2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

Commit message: new board
Parts:
- added G***: LOGO, LOGO, F.Cu at (164.2, 77.8)
Other:
- board text added: "9000"
- board text added: "BROMOTE"
- board text added: "Designed by"
- board text added: "Jared Yang"
- board text added: "THE"
- board text added: "with"
- board text removed: "3-16-26"
- board text removed: "Designed with Zeo by Jared Yang"

Commit message: new boards
Parts:
- Y1: footprint Crystal:Crystal_SMD_3215-2Pin_3.2x1.5mm -> Crystal:Crystal_SMD_HC49-SD
- moved C10 11.5 mm to (162.7, 113.1)
- moved Y1 5.39 mm to (155.0, 113.1), turned to 0 degrees
- moved C11 0.46 mm to (147.5, 115.0), turned to 90 degrees
Routing:
- net GND: track 27.9 -> 17.0 mm
- net Net-(U2-XTAL1): track 5.42 -> 12.3 mm
- net Net-(U2-XTAL2): track 4.99 -> 4.31 mm
- added copper zone on B.Cu, net Net-(U2-XTAL1)
- added copper zone on B.Cu, net Net-(U2-XTAL2)

Commit message: updated
Parts:
- moved J2 0.59 mm to (148.5, 144.3)
Routing:
- net /VBUS: track 28.0 -> 29.8 mm
- net +3V3: track 172.7 -> 173.7 mm
- net GND: vias 12 -> 13
Changed lines of the file:
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@@
 	(footprint "Connector_USB:USB_C_Receptacle_HRO_TYPE-C-31-M-12"
 		(layer "B.Cu")
-		(at 148.51 143.73 180)
+		(at 148.51 144.32 180)
 		(descr "USB Type-C receptacle for USB 2.0 and PD, http://www.krhro.com/uploads/soft/180320/1-1P320120243.pdf")
 		(tags "usb usb-c 2.0 pd")
@@
 	)
 	(segment
+		(start 151.0394 133.28)
+		(end 151.0394 136.082902)
+		(width 0.4)
+		(layer "B.Cu")
+		(net "+3V3")
+	)
+	(segment
 		(start 146.55 116.43)
 		(end 146.55 116.970001)
@@
 	)
 	(segment
-		(start 151.0394 136.082902)
-		(end 151.0394 133.28)
-		(width 0.4)
-		(layer "B.Cu")
-		(net "+3V3")
-	)
-	(segment
 		(start 147.11 119.004999)
 		(end 148.835001 120.73)
@@
 	)
 	(segment
+		(start 158.7144 142.3944)
+		(end 158.7144 143.1675)
+		(width 0.4)
+		(layer "B.Cu")
+		(net "+3V3")
+	)
+	(segment
 		(start 146.86 132.86)
 		(end 150.62 132.86)
@@
 	)
 	(segment
+		(start 158.2 141.88)
+		(end 158.7144 142.3944)
+		(width 0.4)
+		(layer "B.Cu")
+		(net "+3V3")
+	)
+	(segment
 		(start 146.55 116.970001)
 		(end 147.11 117.530001)
@@
 	)
 	(segment
+		(start 151.0394 136.082902)
+		(end 156.836498 141.88)
+		(width 0.4)
+		(layer "B.Cu")
+		(net "+3V3")
+	)
+	(segment
 		(start 144.584999 127.13)
 		(end 143.8475 127.13)
@@
 	)
 	(segment
+		(start 156.836498 141.88)
+		(end 158.2 141.88)
+		(width 0.4)
+		(layer "B.Cu")
+		(net "+3V3")
+	)
+	(segment
 		(start 145.51 129.5925)
 		(end 145.5 129.6025)
@@
 	)
 	(segment
-		(start 158.123998 143.1675)
-		(end 151.0394 136.082902)
-		(width 0.4)
-		(layer "B.Cu")
-		(net "+3V3")
-	)
-	(segment
 		(start 147.83 49.814576)
 		(end 145.554576 49.814576)
@@
 	)
 	(via
+		(at 167.2 142.71)
+		(size 0.6)
+		(drill 0.3)
+		(layers "F.Cu" "B.Cu")
+		(free yes)
+		(net "GND")
+	)
+	(via
 		(at 156.99 130.1)
 		(size 0.6)
@@
 	)
 	(segment
+		(start 150.62 141.4)
+		(end 150.623984 141.4)
+		(width 0.4)
+		(layer "B.Cu")
+		(net "/VBUS")
+	)
+	(segment
+		(start 150.623984 141.4)
+		(end 150.96 141.063984)
+		(width 0.4)
+		(layer "B.Cu")
+		(net "/VBUS")
+	)
+	(segment
 		(start 146.06 139.685)
 		(end 146.06 140.473984)
@@
 	)
 	(segment
-		(start 146.466016 140.88)
-		(end 150.553984 140.88)
+		(start 140.28 123.14)
+		(end 140.27 123.15)
 		(width 0.4)
 		(layer "B.Cu")
@@
 	)
 	(segment
-		(start 140.28 123.14)
-		(end 140.27 123.15)
+		(start 150.96 141.063984)
+		(end 150.96 140.275)
 		(width 0.4)
 		(layer "B.Cu")
@@
 	)
 	(segment
-		(start 146.06 140.473984)
-		(end 146.466016 140.88)
+		(start 146.786016 141.79)
+		(end 150.23 141.79)
 		(width 0.4)
 		(layer "B.Cu")
@@
 	)
 	(segment
+		(start 146.06 141.063984)
+		(end 146.786016 141.79)
+		(width 0.4)
+		(layer "B.Cu")
+		(net "/VBUS")
+	)
+	(segment
+		(start 146.06 140.275)
+		(end 146.06 141.063984)
+		(width 0.4)
+		(layer "B.Cu")
+		(net "/VBUS")
+	)
+	(segment
 		(start 150.96 138.4844)
 		(end 151.6644 137.78)
@@
 	)
 	(segment
-		(start 150.553984 140.88)
-		(end 150.96 140.473984)
+		(start 150.23 141.79)
+		(end 150.62 141.4)
 		(width 0.4)
 		(layer "B.Cu")
@@
 	)
 	(segment
-		(start 162.35 144.905685)
-		(end 160.855685 146.4)
+		(start 136.92 146.55)
+		(end 134.44 144.07)
 		(width 0.2)
 		(layer "B.Cu")
@@
 	)
 	(segment
-		(start 134.44 144.07)
-		(end 134.44 142.13)
+		(start 155.1725 122.33)
+		(end 156.7 122.33)
 		(width 0.2)
 		(layer "B.Cu")
@@
 	)
 	(segment
-		(start 155.1725 122.33)
-		(end 156.7 122.33)
+		(start 162.35 127.98)
+		(end 162.35 144.905685)
 		(width 0.2)
 		(layer "B.Cu")
@@
 	)
 	(segment
-		(start 160.855685 146.4)
-		(end 136.77 146.4)
+		(start 134.44 144.07)
+		(end 134.44 142.13)
 		(width 0.2)
 		(layer "B.Cu")
@@
 	)
 	(segment
-		(start 136.77 146.4)
-		(end 134.44 144.07)
+		(start 162.35 144.905685)
+		(end 160.705685 146.55)
 		(width 0.2)
 		(layer "B.Cu")
@@
 	)
 	(segment
-		(start 134.44 142.13)
-		(end 135.835 140.735)
+		(start 160.705685 146.55)
+		(end 136.92 146.55)
 		(width 0.2)
 		(layer "B.Cu")
@@
 	)
 	(segment
-		(start 156.7 122.33)
-		(end 162.35 127.98)
+		(start 134.44 142.13)
+		(end 135.835 140.735)
 		(width 0.2)
 		(layer "B.Cu")
@@
 	)
 	(segment
-		(start 162.35 127.98)
-		(end 162.35 144.905685)
+		(start 156.7 122.33)
+		(end 162.35 127.98)
 		(width 0.2)
 		(layer "B.Cu")
@@
 		(width 0.2)
 		(layer "B.Cu")
-		(net "/USB_DM")
-	)
-	(segment
-		(start 148.24 139.665)
-		(end 148.26 139.685)
-		(width 0.2)
-		(layer "B.Cu")
