File: ZeoEnvModule/ZeoEnvModule.kicad_pcb (KiCad board)
At the start: 2 copper layers, 19.7 x 32.5 mm, 42 parts, among them J2 USB_C_Receptacle_USB2.0_16P, J3 BATT, SW2 BOOT, SW3 RESET, U2 MCP73871-2CC, U3 AP2112K-3.3, U4 ESP32-S3-WROOM-1, U5 BME280, U6 LSM6DS3

Commit message: updates
Parts:
- added C13: 47uF, Capacitor_SMD:C_1210_3225Metric, B.Cu at (147.7, 117.5)
- added U1: USBLC6-2SC6, Package_TO_SOT_SMD:SOT-23-6, F.Cu at (155.7, 121.5)
- C6: moved to B.Cu
- J3: moved to F.Cu
- moved G*** 10.3 mm to (146.4, 117.2)
- moved R2 1.82 mm to (159.5, 118.7)
- moved R3 1.41 mm to (152.1, 118.8)
- moved R8 0.48 mm to (149.8, 116.0), turned to 45 degrees
- moved R6 0.36 mm to (148.5, 115.3), turned to 135 degrees
Routing:
- net /USB_D+: track 20.1 -> 29.6 mm
- net /Power Supply/VBUS: track 37.1 -> 43.7 mm, vias 0 -> 1
- net /USB_D-: track 25.0 -> 30.9 mm, vias 3 -> 4
- net GND: track 7.26 -> 8.98 mm, vias 7 -> 11
- net Net-(J2-CC1): track 2.58 -> 3.80 mm
- net Net-(J2-CC2): track 2.57 -> 3.77 mm
- net /MCU/EN: track 27.1 -> 25.9 mm
- net Net-(U2-PROG3): track 1.52 -> 2.33 mm
