File: ZeoEnvModule/power_supply.kicad_sch (KiCad schematic)
At the start: 23 parts, among them J2 USB_C_Receptacle_USB2.0_16P, J3 BATT, U2 MCP73871-2CC, U3 AP2112K-3.3

Commit message: updates
Parts:
- added C13: 47uF, Capacitor_SMD:C_1210_3225Metric, symbol Device:C
- added U1: USBLC6-2SC6, Package_TO_SOT_SMD:SOT-23-6, symbol Power_Protection:USBLC6-2SC6
Connections:
- net GND: now also C13.1, U1.2 (GND)
- net USB_D+: now also U1.3 (I/O2), U1.4 (I/O2)
- net USB_D-: now also U1.1 (I/O1), U1.6 (I/O1)
- net VBAT: now also C13.2
- net VBUS: now also U1.5 (VBUS)
Other:
- moved on the sheet: C2, C3, C4, C5, D2, D3, D4, J2, J3, R10, R11, R12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
