File: demo_board/ZeoDevBoard.kicad_pcb (KiCad board)
At the start: 2 copper layers, 20.1 x 31 mm, 36 parts, among them J2 USB_C_Receptacle_USB2.0_14P, J3 BATTERY, SW1 RESET, SW2 BOOT, U1 ESP32-S3-WROOM-1, U2 USBLC6-2SC6, U3 MCP73871-2CC, U4 AP2112K-3.3, U5 BME280, U6 LSM6DS3

Commit message: updated
Parts:
- moved J2 34.3 mm to (153.5, 108.3)
- moved R3 33.7 mm to (151.4, 108.2)
- moved U2 33.7 mm to (154.1, 108.8)
- moved R2 33.7 mm to (152.8, 101.1)
- moved R7 33.6 mm to (147.0, 94.1)
- moved R5 33.3 mm to (146.5, 95.5)
- moved C2 33.3 mm to (143.8, 97.6)
- moved C4 33.3 mm to (155.8, 98.2)
- moved C5 33.3 mm to (143.0, 102.2)
- moved J3 33.3 mm to (143.9, 105.7)
- moved R11 33.3 mm to (142.8, 107.3)
- moved R12 33.3 mm to (146.2, 107.3)
- moved R4 33.3 mm to (155.3, 95.8)
- moved R6 33.3 mm to (155.3, 94.3)
- moved U5 33.3 mm to (153.2, 86.2)
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Routing:
- net /Power Supply/USB_DP_RAW: track 5.24 -> 18.2 mm, vias 1 -> 2
- net GND: track 12.8 -> 4.87 mm, vias 11 -> 12
- net VBUS: track 37.9 -> 33.2 mm
- net /USB_DP: track 17.9 -> 21.0 mm
- net /Power Supply/USB_DN_RAW: track 19.9 -> 18.2 mm
- net /SCL: track 27.2 -> 28.8 mm
- net +3V3: track 67.7 -> 69.0 mm
- net Net-(D4-K): track 7.39 -> 8.14 mm
- net Net-(D3-K): track 9.18 -> 9.90 mm
- net Net-(J2-CC1): track 1.74 -> 2.44 mm
- net Net-(U3-PROG2): track 1.35 -> 1.92 mm
- net /IMU_INT2: track 17.8 -> 17.4 mm, vias 3 -> 1
- net /IMU_INT1: track 19.3 -> 19.0 mm, vias 2 -> 1
Other:
- board text added: "P"
- board text removed: "PG"
