File: zeo1_devboard/mcu.kicad_sch (KiCad schematic)
At the start: 31 parts, among them J4 Micro_SD, Q2 BC817, Q3 BC817, U5 USBLC6-2SC6, U6 CP2102N-QFN24, U7 ESP32-C3, U8 ANT3216LL00R2400A, U9 W25Q32JVSS, Y1 40MHz

Commit message: new demo board
Parts:
- removed C15: 0.1uF, Capacitor_SMD:C_0402_1005Metric, symbol Device:C
Connections:
- net +3V3: no longer J4.6 (VSS)
- net +5V_USB: now also U5.5 (VBUS), U6.8 (VBUS)
- net BOOT: now also R23.1; no longer R25.1
- net EN: now also R25.1; no longer R23.1
- net GND: now also J4.6 (VSS); no longer Q2.2 (E), Q3.2 (E)
- net ~DTR: now also Q3.2 (E)
- net ~RTS: now also Q2.2 (E)
