File: zeo1_devboard/sensors.kicad_sch (KiCad schematic)
At the start: 14 parts, among them Q1 TEMT6000, U3 BME280, U4 MAX4466

Commit message: new demo board
Parts:
- R17: value 1k -> 10k
- R18: value 1M -> 220k
Other:
- moved on the sheet: R18
Changed lines of the file:
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@@
-	)
-	(junction
-		(at 213.36 113.03)
-		(diameter 0)
-		(color 0 0 0 0)
 	)
 	(junction
@@
 	)
 	(junction
-		(at 71.12 119.38)
-		(diameter 0)
-		(color 0 0 0 0)
-	)
-	(junction
 		(at 138.43 101.6)
 		(diameter 0)
@@
 		(color 0 0 0 0)
 	)
+	(junction
+		(at 212.09 113.03)
+		(diameter 0)
+		(color 0 0 0 0)
+	)
 	(wire
 		(pts
@@
 	(wire
 		(pts
-			(xy 222.25 119.38) (xy 213.36 119.38)
-		)
-		(stroke
-			(width 0)
-			(type default)
-		)
-	)
-	(wire
-		(pts
-			(xy 213.36 113.03) (xy 213.36 119.38)
-		)
-		(stroke
-			(width 0)
-			(type default)
-		)
-	)
-	(wire
-		(pts
 			(xy 204.47 102.87) (xy 190.5 102.87)
 		)
@@
 	(wire
 		(pts
-			(xy 72.39 120.65) (xy 72.39 119.38)
+			(xy 212.09 115.57) (xy 223.52 115.57)
 		)
 		(stroke
@@
 	(wire
 		(pts
-			(xy 218.44 113.03) (xy 218.44 114.3)
-		)
-		(stroke
-			(width 0)
-			(type default)
-		)
-	)
-	(wire
-		(pts
-			(xy 209.55 113.03) (xy 213.36 113.03)
+			(xy 218.44 113.03) (xy 218.44 124.46)
+		)
+		(stroke
+			(width 0)
+			(type default)
+		)
+	)
+	(wire
+		(pts
+			(xy 209.55 113.03) (xy 212.09 113.03)
+		)
+		(stroke
+			(width 0)
+			(type default)
+		)
+	)
+	(wire
+		(pts
+			(xy 76.2 120.65) (xy 76.2 119.38)
 		)
 		(stroke
@@
 	(wire
 		(pts
-			(xy 213.36 107.95) (xy 213.36 113.03)
-		)
-		(stroke
-			(width 0)
-			(type default)
-		)
-	)
-	(wire
-		(pts
 			(xy 218.44 85.09) (xy 218.44 83.82)
 		)
@@
 	(wire
 		(pts
-			(xy 76.2 119.38) (xy 76.2 120.65)
-		)
-		(stroke
-			(width 0)
-			(type default)
-		)
-	)
-	(wire
-		(pts
 			(xy 213.36 102.87) (xy 212.09 102.87)
 		)
@@
 	(wire
 		(pts
+			(xy 212.09 113.03) (xy 212.09 107.95)
+		)
+		(stroke
+			(width 0)
+			(type default)
+		)
+	)
+	(wire
+		(pts
 			(xy 144.78 101.6) (xy 138.43 101.6)
 		)
@@
 	(wire
 		(pts
-			(xy 76.2 120.65) (xy 72.39 120.65)
-		)
-		(stroke
-			(width 0)
-			(type default)
-		)
-	)
-	(wire
-		(pts
 			(xy 76.2 88.9) (xy 76.2 87.63)
 		)
@@
 	(wire
 		(pts
+			(xy 213.36 107.95) (xy 212.09 107.95)
+		)
+		(stroke
+			(width 0)
+			(type default)
+		)
+	)
+	(wire
+		(pts
 			(xy 90.17 106.68) (xy 88.9 106.68)
 		)
@@
 	(wire
 		(pts
-			(xy 72.39 119.38) (xy 71.12 119.38)
-		)
-		(stroke
-			(width 0)
-			(type default)
-		)
-	)
-	(wire
-		(pts
 			(xy 138.43 111.76) (xy 138.43 113.03)
 		)
@@
 	(wire
 		(pts
-			(xy 231.14 119.38) (xy 231.14 105.41)
+			(xy 231.14 115.57) (xy 231.14 105.41)
 		)
 		(stroke
@@
 	(wire
 		(pts
-			(xy 229.87 119.38) (xy 231.14 119.38)
+			(xy 212.09 115.57) (xy 212.09 113.03)
 		)
 		(stroke
@@
 	(symbol
 		(lib_id "Device:R")
-		(at 226.06 119.38 90)
+		(at 227.33 115.57 90)
 		(unit 1)
 		(body_style 1)
@@
 		(dnp no)
 		(property "Reference" "R18"
-			(at 226.06 117.094 90)
-			(show_name no)
-			(do_not_autoplace no)
-			(effects
-				(font
-					(size 1.27 1.27)
-				)
-			)
-		)
-		(property "Value" "1M"
-			(at 226.06 119.38 90)
+			(at 227.33 113.284 90)
+			(show_name no)
+			(do_not_autoplace no)
+			(effects
+				(font
+					(size 1.27 1.27)
+				)
+			)
+		)
+		(property "Value" "220k"
+			(at 227.33 115.57 90)
 			(show_name no)
 			(do_not_autoplace no)
@@
 		)
 		(property "Footprint" "Resistor_SMD:R_0402_1005Metric"
-			(at 220.98 118.618 90)
+			(at 222.25 114.808 90)
 			(hide yes)
 			(show_name no)
@@
 		)
 		(property "Datasheet" ""
-			(at 220.98 116.84 0)
+			(at 222.25 113.03 0)
 			(hide yes)
 			(show_name no)
@@
 		)
 		(property "Description" "Resistor"
-			(at 220.98 116.84 0)
-			(hide yes)
-			(show_name no)
-			(do_not_autoplace no)
-			(effects
-				(font
-					(size 1.27 1.27)
-				)
-			)
+			(at 222.25 113.03 0)
+			(hide yes)
+			(show_name no)
+			(do_not_autoplace no)
+			(effects
+				(font
+					(size 1.27 1.27)
+				)
+			)
+		)
+		(pin "1"
 		)
 		(pin "2"
-		)
-		(pin "1"
 		)
 		(instances
@@
 			)
 		)
-		(property "Value" "1k"
+		(property "Value" "10k"
 			(at 205.74 113.03 90)
 			(show_name no)
@@
 			)
 		)
+		(pin "2"
+		)
 		(pin "1"
-		)
-		(pin "2"
 		)
 		(instances
@@
 	(symbol
 		(lib_id "power:GND")
-		(at 218.44 114.3 0)
+		(at 218.44 124.46 0)
 		(unit 1)
 		(body_style 1)
@@
 		(dnp no)
 		(property "Reference" "#PWR025"
-			(at 218.44 120.65 0)
+			(at 218.44 130.81 0)
 			(hide yes)
 			(show_name no)
@@
 		)
 		(property "Value" "GND"
-			(at 218.44 118.11 0)
+			(at 218.44 128.27 0)
 			(show_name no)
 			(do_not_autoplace no)
@@
 		)
 		(property "Footprint" ""
-			(at 218.44 114.3 0)
+			(at 218.44 124.46 0)
 			(hide yes)
 			(show_name no)
@@
 		)
 		(property "Datasheet" ""
-			(at 218.44 114.3 0)
+			(at 218.44 124.46 0)
 			(hide yes)
 			(show_name no)
@@
 		)
 		(property "Description" "Power symbol creates a global label with name \"GND\" , ground"
-			(at 218.44 114.3 0)
+			(at 218.44 124.46 0)
 			(hide yes)
 			(show_name no)
@@
 					(unit 1)
 				)
+			)
+		)
+	)
+	(symbol
+		(lib_id "power:GND")
+		(at 76.2 120.65 0)
+		(unit 1)
+		(body_style 1)
+		(exclude_from_sim no)
+		(in_bom yes)
+		(on_board yes)
+		(in_pos_files yes)
+		(dnp no)
+		(property "Reference" "#PWR033"
+			(at 76.2 127 0)
+			(hide yes)
+			(show_name no)
+			(do_not_autoplace no)
+			(effects
+				(font
+					(size 1.27 1.27)
+				)
+			)
+		)
+		(property "Value" "GND"
+			(at 76.2 124.46 0)
+			(show_name no)
+			(do_not_autoplace no)
+			(effects
+				(font
+					(size 1.27 1.27)
+				)
+			)
+		)
+		(property "Footprint" ""
+			(at 76.2 120.65 0)
+			(hide yes)
+			(show_name no)
+			(do_not_autoplace no)
+			(effects
+				(font
+					(size 1.27 1.27)
+				)
+			)
+		)
+		(property "Datasheet" ""
+			(at 76.2 120.65 0)
+			(hide yes)
+			(show_name no)
+			(do_not_autoplace no)
+			(effects
+				(font
+					(size 1.27 1.27)
+				)
+			)
+		)
+		(property "Description" "Power symbol creates a global label with name \"GND\" , ground"
+			(at 76.2 120.65 0)
+			(hide yes)
+			(show_name no)
+			(do_not_autoplace no)
+			(effects
+				(font
+					(size 1.27 1.27)
+				)
+			)
+		)
+		(pin "1"
+		)
+		(instances
+			(project "zeo1_devboard"
+				(path "/1d9d5540-a5fb-439a-a7fc-dd6397c3c196/2c52d406-dcf9-43e0-9fef-72b1ad65cf4c"
+					(reference "#PWR033")
+					(unit 1)
+				)
