File: zeo1_devboard/zeo1_devboard.kicad_pcb (KiCad board)
At the start: 4 copper layers, 25.4 x 25.4 mm, 92 parts, among them J1 USB_C_Receptacle_USB2.0_14P, J2 JST-PH Battery, J3 OLED Display, J4 Micro_SD, Q1 TEMT6000, Q2 BC817, Q3 BC817, SW1 BOOT, SW2 RESET, U1 AP2112K-3.3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

Commit message: new demo board
Parts:
- removed C15: 0.1uF, Capacitor_SMD:C_0402_1005Metric
- removed R9: 100k, Resistor_SMD:R_0402_1005Metric
- R17: value 1k -> 10k
- R18: value 1M -> 220k
Connections:
- J1 pad B6: unconnected-(J1-D+-PadB6) -> /USB_DP
- J1 pad B7: unconnected-(J1-D--PadB7) -> /USB_DN
- J4 pad 6: /+3V3 -> GND
- Q2 pad 2: GND -> /MCU/~RTS
- Q3 pad 2: GND -> /MCU/~DTR
- R23 pad 1: /EN -> /BOOT
- R25 pad 1: /BOOT -> /EN
- R4 pad 1: GND -> /+5V_USB
- R7 pad 1: /+5V_USB -> GND
- U2 pad 2: Net-(U2-VPCC) -> /+5V_USB
- U5 pad 5: Net-(U5-VBUS) -> /+5V_USB
- U6 pad 8: Net-(U5-VBUS) -> /+5V_USB
Routing:
- net GND: track 21.3 -> 28.9 mm
- net /+5V_USB: track 38.0 -> 43.0 mm
- net Net-(U5-VBUS): track 3.36 -> 0.00 mm
- net Net-(U2-VPCC): track 1.62 -> 0.00 mm
- net /EN: vias 4 -> 3
- net /+3V3: vias 17 -> 16
