File: zeo1_devboard/zeo1_devboard.kicad_sch (KiCad schematic)
At the start: 30 parts, among them J1 USB_C_Receptacle_USB2.0_14P, J2 JST-PH Battery, U1 AP2112K-3.3, U2 MCP73871

Commit message: new demo board
Parts:
- removed R9: 100k, Resistor_SMD:R_0402_1005Metric, symbol Device:R
Connections:
- net +5V_USB: now also R4.1, U2.2 (VPCC); no longer R7.1
- net GND: now also R7.1; no longer R4.1
- net USB_DN: now also J1.B7 (D-)
- net USB_DP: now also J1.B6 (D+)
- no-connect marks 2 -> 0
