File: zeo1.2_devboard/mcu.kicad_sch (KiCad schematic)
At the start: 30 parts, among them J4 Micro_SD, Q2 BC817, Q3 BC817, U10 ESP32-S3, U5 USBLC6-2SC6, U6 CP2102N-QFN24, U7 W25Q128JVSIQ, U8 ANT3216LL00R2400A, Y1 40MHz

Commit message: new demo board
Parts:
- added C12: 4.7uF, symbol Device:C
Connections:
- net +3V3: no longer C19.2
- net +5V_USB: now also U5.5 (VBUS), U6.8 (VBUS), C12.2
- net GND: now also C12.1
Changed lines of the file:
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@@
 		(color 0 0 0 0)
 	)
+	(junction
+		(at 31.75 52.07)
+		(diameter 0)
+		(color 0 0 0 0)
+	)
 	(no_connect
 		(at 66.04 57.15)
@@
 	(wire
 		(pts
-			(xy 50.8 33.02) (xy 50.8 34.29)
-		)
-		(stroke
-			(width 0)
-			(type default)
-		)
-	)
-	(wire
-		(pts
 			(xy 212.09 143.51) (xy 195.58 143.51)
 		)
@@
 	(wire
 		(pts
-			(xy 55.88 33.02) (xy 55.88 34.29)
+			(xy 45.72 21.59) (xy 45.72 20.32)
 		)
 		(stroke
@@
 	(wire
 		(pts
-			(xy 195.58 143.51) (xy 189.23 143.51)
+			(xy 55.88 33.02) (xy 55.88 34.29)
 		)
 		(stroke
@@
 	(wire
 		(pts
-			(xy 138.43 66.04) (xy 138.43 62.23)
+			(xy 195.58 143.51) (xy 189.23 143.51)
 		)
 		(stroke
@@
 	(wire
 		(pts
-			(xy 24.13 57.15) (xy 26.67 57.15)
+			(xy 138.43 66.04) (xy 138.43 62.23)
 		)
 		(stroke
@@
 	(wire
 		(pts
-			(xy 90.17 187.96) (xy 90.17 185.42)
+			(xy 24.13 57.15) (xy 26.67 57.15)
 		)
 		(stroke
@@
 	(wire
 		(pts
-			(xy 31.75 52.07) (xy 40.64 52.07)
+			(xy 90.17 187.96) (xy 90.17 185.42)
 		)
 		(stroke
@@
 	(wire
 		(pts
+			(xy 31.75 52.07) (xy 40.64 52.07)
+		)
+		(stroke
+			(width 0)
+			(type default)
+		)
+	)
+	(wire
+		(pts
 			(xy 45.72 177.8) (xy 46.99 177.8)
 		)
@@
 	(wire
 		(pts
-			(xy 59.69 29.21) (xy 53.34 29.21)
+			(xy 53.34 29.21) (xy 66.04 29.21)
 		)
 		(stroke
@@
 	(wire
 		(pts
+			(xy 45.72 29.21) (xy 50.8 29.21)
+		)
+		(stroke
+			(width 0)
+			(type default)
+		)
+	)
+	(wire
+		(pts
 			(xy 45.72 172.72) (xy 46.99 172.72)
 		)
@@
 	(wire
 		(pts
+			(xy 31.75 50.8) (xy 31.75 52.07)
+		)
+		(stroke
+			(width 0)
+			(type default)
+		)
+	)
+	(wire
+		(pts
 			(xy 36.83 59.69) (xy 38.1 59.69)
 		)
@@
 	(wire
 		(pts
+			(xy 50.8 29.21) (xy 50.8 34.29)
+		)
+		(stroke
+			(width 0)
+			(type default)
+		)
+	)
+	(wire
+		(pts
 			(xy 212.09 130.81) (xy 212.09 143.51)
 		)
@@
 	(wire
 		(pts
-			(xy 49.53 29.21) (xy 53.34 29.21)
-		)
-		(stroke
-			(width 0)
-			(type default)
-		)
-	)
-	(wire
-		(pts
 			(xy 114.3 151.13) (xy 114.3 152.4)
 		)
@@
 	)
 	(label "+3V3"
-		(at 49.53 29.21 180)
+		(at 66.04 29.21 0)
 		(effects
 			(font
@@
 				(line_spacing 0)
 			)
-			(justify right bottom)
+			(justify left bottom)
 		)
 	)
@@
 		)
 	)
+	(hierarchical_label "+5V_USB"
+		(shape input)
+		(at 31.75 50.8 180)
+		(effects
+			(font
+				(size 1.27 1.27)
+				(line_spacing 0)
+			)
+			(justify right bottom)
+		)
+	)
 	(hierarchical_label "I2S_SD"
 		(shape input)
@@
 		(dnp no)
 		(property "Reference" "U5"
-			(at 15.494 50.292 0)
+			(at 14.986 64.77 0)
 			(show_name no)
 			(do_not_autoplace no)
@@
 		)
 		(property "Value" "USBLC6-2SC6"
-			(at 15.24 52.324 0)
+			(at 14.732 66.802 0)
 			(show_name no)
 			(do_not_autoplace no)
@@
 	(symbol
 		(lib_id "power:GND")
+		(at 45.72 20.32 180)
+		(unit 1)
+		(body_style 1)
+		(exclude_from_sim no)
+		(in_bom yes)
+		(on_board yes)
+		(in_pos_files yes)
+		(dnp no)
+		(property "Reference" "#PWR073"
+			(at 45.72 13.97 0)
+			(hide yes)
+			(show_name no)
+			(do_not_autoplace no)
+			(effects
+				(font
+					(size 1.27 1.27)
+				)
+			)
+		)
+		(property "Value" "GND"
+			(at 45.72 16.51 0)
+			(show_name no)
+			(do_not_autoplace no)
+			(effects
+				(font
+					(size 1.27 1.27)
+				)
+			)
+		)
+		(property "Footprint" ""
+			(at 45.72 20.32 0)
+			(hide yes)
+			(show_name no)
+			(do_not_autoplace no)
+			(effects
+				(font
+					(size 1.27 1.27)
+				)
+			)
+		)
+		(property "Datasheet" ""
+			(at 45.72 20.32 0)
+			(hide yes)
+			(show_name no)
+			(do_not_autoplace no)
+			(effects
+				(font
+					(size 1.27 1.27)
+				)
+			)
+		)
+		(property "Description" "Power symbol creates a global label with name \"GND\" , ground"
+			(at 45.72 20.32 0)
+			(hide yes)
+			(show_name no)
+			(do_not_autoplace no)
+			(effects
+				(font
+					(size 1.27 1.27)
+				)
+			)
+		)
+		(pin "1"
+		)
+		(instances
+			(project ""
+				(path "/1d9d5540-a5fb-439a-a7fc-dd6397c3c196/0bb7f993-a23f-4f29-8212-e276001f7304"
+					(reference "#PWR073")
+					(unit 1)
+				)
+			)
+		)
+	)
+	(symbol
+		(lib_id "power:GND")
 		(at 31.75 67.31 0)
 		(unit 1)
@@
 					(unit 1)
 				)
+			)
+		)
+	)
+	(symbol
+		(lib_id "Device:C")
+		(at 45.72 25.4 0)
+		(unit 1)
+		(body_style 1)
+		(exclude_from_sim no)
+		(in_bom yes)
+		(on_board yes)
+		(in_pos_files yes)
+		(dnp no)
+		(property "Reference" "C12"
+			(at 46.355 22.86 0)
+			(show_name no)
+			(do_not_autoplace no)
+			(effects
+				(font
+					(size 1.27 1.27)
+				)
+				(justify left)
+			)
+		)
+		(property "Value" "4.7uF"
+			(at 46.355 27.94 0)
+			(show_name no)
+			(do_not_autoplace no)
+			(effects
+				(font
+					(size 1.27 1.27)
+				)
+				(justify left)
+			)
+		)
+		(property "Footprint" ""
+			(at 46.6852 29.21 0)
+			(hide yes)
+			(show_name no)
+			(do_not_autoplace no)
+			(effects
+				(font
+					(size 1.27 1.27)
+				)
+			)
+		)
+		(property "Datasheet" ""
+			(at 45.72 25.4 0)
+			(hide yes)
+			(show_name no)
+			(do_not_autoplace no)
+			(effects
+				(font
+					(size 1.27 1.27)
+				)
+			)
+		)
+		(property "Description" "Unpolarized capacitor"
+			(at 45.72 25.4 0)
+			(hide yes)
+			(show_name no)
+			(do_not_autoplace no)
+			(effects
+				(font
+					(size 1.27 1.27)
+				)
+			)
+		)
+		(pin "2"
+		)
+		(pin "1"
+		)
+		(instances
+			(project ""
+				(path "/1d9d5540-a5fb-439a-a7fc-dd6397c3c196/0bb7f993-a23f-4f29-8212-e276001f7304"
+					(reference "C12")
+					(unit 1)
+				)

Commit message: new boards
Parts:
- C12: footprint (none) -> Capacitor_SMD:C_0805_2012Metric
Connections:
- net +3V3: now also C19.2
Changed lines of the file:
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@@
 	)
 	(junction
-		(at 38.1 170.18)
+		(at 59.69 29.21)
 		(diameter 0)
 		(color 0 0 0 0)
 	)
 	(junction
-		(at 163.83 62.23)
+		(at 38.1 170.18)
 		(diameter 0)
 		(color 0 0 0 0)
 	)
 	(junction
-		(at 114.3 140.97)
+		(at 163.83 62.23)
 		(diameter 0)
 		(color 0 0 0 0)
 	)
 	(junction
-		(at 53.34 29.21)
+		(at 114.3 140.97)
 		(diameter 0)
 		(color 0 0 0 0)
@@
 	)
 	(junction
+		(at 53.34 29.21)
+		(diameter 0)
+		(color 0 0 0 0)
+	)
+	(junction
 		(at 212.09 143.51)
 		(diameter 0)
@@
 	(wire
 		(pts
-			(xy 53.34 29.21) (xy 66.04 29.21)
+			(xy 53.34 29.21) (xy 59.69 29.21)
 		)
 		(stroke
@@
 	(wire
 		(pts
+			(xy 59.69 29.21) (xy 66.04 29.21)
+		)
+		(stroke
+			(width 0)
+			(type default)
+		)
+	)
+	(wire
+		(pts
 			(xy 151.13 66.04) (xy 152.4 66.04)
 		)
@@
 			)
 		)
-		(property "Footprint" ""
+		(property "Footprint" "Capacitor_SMD:C_0805_2012Metric"
 			(at 46.6852 29.21 0)
 			(hide yes)
