File: zeo1.2_devboard/zeo1.2_devboard.kicad_sch (KiCad schematic)
At the start: 30 parts, among them J1 USB_C_Receptacle_USB2.0_14P, J2 JST-PH Battery, U1 AP2112K-3.3, U2 MCP73871

Commit message: new demo board
Parts:
- added C11: 4.7uF, symbol Device:C
- C6: value 1uF -> 4.7uF
Connections:
- net +5V_USB: now also R4.1; no longer R7.1
- net GND: now also R7.1, C11.2; no longer R4.1
- net VBAT: now reaches J2.1 (Pin_1), U2.14 (V_{BAT}), U2.15 (V_{BAT}), U2.16 (V_{BAT_SENSE})
- net VBAT: now also C11.1

Commit message: new boards
Parts:
- C11: footprint (none) -> Capacitor_SMD:C_0805_2012Metric
- J1: footprint Connector_USB:USB_C_Receptacle_Amphenol_12401610E4-2A_CircularHoles -> Connector_USB:USB_C_Receptacle_GCT_USB4085
- J2: footprint Connector_JST:JST_ZH_B2B-ZR_1x02_P1.50mm_Vertical -> Connector_JST:JST_PH_B2B-PH-K_1x02_P2.00mm_Vertical
Changed lines of the file:
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@@
 			)
 		)
-		(property "Footprint" "Connector_USB:USB_C_Receptacle_Amphenol_12401610E4-2A_CircularHoles"
+		(property "Footprint" "Connector_USB:USB_C_Receptacle_GCT_USB4085"
 			(at 41.91 50.8 0)
 			(hide yes)
@@
 			)
 		)
-		(property "Footprint" ""
+		(property "Footprint" "Capacitor_SMD:C_0805_2012Metric"
 			(at 102.5652 139.7 0)
 			(hide yes)
@@
 			)
 		)
-		(property "Footprint" "Connector_JST:JST_ZH_B2B-ZR_1x02_P1.50mm_Vertical"
+		(property "Footprint" "Connector_JST:JST_PH_B2B-PH-K_1x02_P2.00mm_Vertical"
 			(at 149.86 45.72 0)
 			(hide yes)
