File: zeo1.2_devboard/zeo1.2_devboard.kicad_pcb (KiCad board)
At the start: 4 copper layers, 25.4 x 25.4 mm, 97 parts, among them J1 USB_C_Receptacle_USB2.0_14P, J2 JST-PH Battery, J4 Micro_SD, Q2 BC817, Q3 BC817, U1 AP2112K-3.3, U10 ESP32-S3, U11 LSM6DS3, U12 BMM150, U13 W3011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

Commit message: updates
Routing:
- net GND: track 21.9 -> 19.5 mm
- net /MISO_DO: track 16.7 -> 17.3 mm

Commit message: new boards
Parts:
- removed G***: LOGO, LOGO
- C6: value 1uF -> 4.7uF
- renumbered B to SW1, R to SW2
Connections:
- net Net-(J2-Pin_1) renamed /VBAT
- C19 pad 2: +3V3 -> unconnected-(C19-Pad2)
- R4 pad 1: GND -> /+5V_USB
- R7 pad 1: /+5V_USB -> GND
- U5 pad 5: Net-(U5-VBUS) -> /+5V_USB
- U6 pad 8: Net-(U5-VBUS) -> /+5V_USB
Routing:
- net +3V3: track 103.9 -> 0.00 mm, vias 18 -> 0
- net /SCL: track 58.6 -> 0.00 mm, vias 7 -> 0
- net /+5V_USB: track 46.2 -> 0.00 mm, vias 6 -> 0
- net /SDA: track 43.9 -> 0.00 mm, vias 6 -> 0
- net /EN: track 26.4 -> 0.00 mm, vias 2 -> 0
- net Net-(D2-K): track 22.7 -> 0.00 mm, vias 2 -> 0
- net Net-(D4-K): track 22.3 -> 0.00 mm, vias 2 -> 0
- net GND: track 19.5 -> 0.00 mm, vias 23 -> 0
- net /MCU/~DTR: track 18.1 -> 0.00 mm, vias 2 -> 0
- net /TX_RX: track 17.5 -> 0.00 mm, vias 2 -> 0
- net /GPS_TX: track 17.3 -> 0.00 mm, vias 2 -> 0
- net /MISO_DO: track 17.3 -> 0.00 mm, vias 2 -> 0
- net Net-(D3-K): track 17.2 -> 0.00 mm, vias 2 -> 0
- net /MCU/~RTS: track 17.2 -> 0.00 mm, vias 2 -> 0
- net /RX_TX: track 17.0 -> 0.00 mm, vias 2 -> 0
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
Commit message: new boards
Parts:
- removed TP2, TP3, TP4, TP6, TP7, TP8, TP9: TestPoint, TestPoint:TestPoint_Pad_1.0x1.0mm
- added C11: 4.7uF, Capacitor_SMD:C_0805_2012Metric, F.Cu at (138.3, 99.3)
- added C12: 4.7uF, Capacitor_SMD:C_0805_2012Metric, B.Cu at (151.0, 98.6)
- added G***: LOGO, LOGO, F.Cu at (159.2, 89.6)
- C10, C38, Q2, Q3, R16, R22, R23, R24, R25: moved to B.Cu
- C19, C21, C26, C32, C33, C34, C9, F1, R1, R2, U1, U11, U12: moved to F.Cu
- J1: footprint Connector_USB:USB_C_Receptacle_Amphenol_12401610E4-2A_CircularHoles -> Connector_USB:USB_C_Receptacle_GCT_USB4085
- J2: footprint Connector_JST:JST_ZH_B2B-ZR_1x02_P1.50mm_Vertical -> Connector_JST:JST_PH_B2B-PH-K_1x02_P2.00mm_Vertical
- moved C17 22.8 mm to (152.5, 111.5), turned to 90 degrees
- moved R13 19.0 mm to (143.1, 94.2)
- moved D3 19.0 mm to (142.6, 95.6), turned to 90 degrees
- moved D2 19.0 mm to (144.5, 95.6), turned to 90 degrees
- moved R12 19.0 mm to (141.2, 95.1)
- moved D4 18.9 mm to (143.6, 95.6), turned to 90 degrees
- moved U6 18.3 mm to (154.3, 107.2), turned to 0 degrees
- moved C9 17.4 mm to (144.7, 89.4), turned to 90 degrees
- moved D5 17.3 mm to (161.9, 92.5), turned to -90 degrees
- moved R11 17.3 mm to (146.1, 95.1), turned to 180 degrees
- moved R7 16.4 mm to (141.2, 96.1), turned to 0 degrees
- moved D6 16.3 mm to (161.0, 92.5), turned to -90 degrees
- moved U5 16.1 mm to (149.6, 111.0), turned to 0 degrees
- moved C18 15.7 mm to (148.1, 108.5), turned to -90 degrees
- moved R20 15.6 mm to (161.9, 94.4), turned to 90 degrees
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Connections:
- C19 pad 2: unconnected-(C19-Pad2) -> +3V3
Routing:
- net /BOOT: track 0.00 -> 37.2 mm, vias 0 -> 2
- net /RX_TX: track 0.00 -> 33.3 mm, vias 0 -> 2
- net /EN: track 0.00 -> 33.2 mm, vias 0 -> 2
- net /SCL: track 0.00 -> 29.1 mm, vias 0 -> 4
- net /SDA: track 0.00 -> 28.8 mm, vias 0 -> 5
- net +3V3: track 0.00 -> 24.9 mm, vias 0 -> 17
- net /I2S_SD: track 0.00 -> 23.0 mm, vias 0 -> 2
- net /TX_RX: track 0.00 -> 22.4 mm, vias 0 -> 2
- net GND: track 0.00 -> 22.2 mm, vias 0 -> 23
- net /MCU/FLASH_CS: track 0.00 -> 18.9 mm, vias 0 -> 2
- net /GPS_RX: track 0.00 -> 18.6 mm, vias 0 -> 2
- net /GPS_TX: track 0.00 -> 18.0 mm, vias 0 -> 2
- net /MCU/~RTS: track 0.00 -> 17.1 mm, vias 0 -> 2
- net /MISO_DO: track 0.00 -> 16.4 mm, vias 0 -> 1
- net /MCU/FLASH_Q: track 0.00 -> 14.7 mm, vias 0 -> 2
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- added copper zone on In2.Cu, net +3V3
- added copper zone on F.Cu, net /+5V
- added copper zone on In2.Cu, net /+5V_USB
- added copper zone on F.Cu, net /MCU/VDD_SPI
- removed copper zone on F.Cu, net /BOOT
- removed copper zone on In2.Cu, net GND

Commit message: updated
Parts:
- moved D5 1.26 mm to (162.1, 93.8)
- moved D6 1.26 mm to (161.1, 93.8)
- moved D7 1.26 mm to (160.2, 93.8)
- moved R20 1.26 mm to (162.0, 95.6)
- moved R21 1.26 mm to (161.1, 95.6)
- moved R26 1.26 mm to (160.2, 95.6)
- moved C37 0.40 mm to (158.6, 93.5)
Routing:
- net GND: track 22.2 -> 18.7 mm
- net /LED_R: track 6.35 -> 8.48 mm

Commit message: 1.2 updates
Parts:
- C12: moved to F.Cu
- moved C12 8.84 mm to (150.6, 107.5), turned to -90 degrees
- moved C18 2.04 mm to (146.5, 109.9), turned to 0 degrees
- moved C2 1.61 mm to (146.5, 106.2), turned to 0 degrees
- moved C19 1.17 mm to (148.4, 107.6)
- moved C14 0.84 mm to (144.5, 109.8)
- moved C13 0.72 mm to (140.6, 109.7)
- moved R19 0.63 mm to (142.6, 109.7)
- moved R4 0.39 mm to (147.0, 98.8), turned to -100 degrees
- moved R9 0.08 mm to (146.1, 100.7), turned to 55 degrees
Routing:
- net /RX_TX: track 33.3 -> 11.4 mm
- net /I2S_SD: track 23.0 -> 14.8 mm
- net /TX_RX: track 22.5 -> 15.5 mm
- net +3V3: track 25.0 -> 18.1 mm, vias 17 -> 16
- net /MCU/FLASH_D: track 9.83 -> 15.2 mm
- net /MCU/~RTS: track 17.1 -> 22.1 mm
- net /MCU/FLASH_HD: track 8.67 -> 13.5 mm
- net /EN: track 33.2 -> 28.9 mm
- net /BOOT: track 37.2 -> 33.0 mm
- net /LED_R: track 8.48 -> 5.21 mm, vias 2 -> 0
- net GND: track 18.7 -> 21.8 mm, vias 23 -> 22
- net /MCU/FLASH_CS: track 18.9 -> 16.5 mm
- net /+5V_USB: track 4.39 -> 6.63 mm
- net /SCL: track 29.1 -> 27.0 mm
- net /LED_B: track 4.49 -> 2.46 mm, vias 2 -> 0
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- added copper zone on F.Cu, net /EN

Commit message: updated
Parts:
- R20, R21, R26: moved to B.Cu
- moved C37 10.2 mm to (148.7, 96.1), turned to 145 degrees
- moved C22 1.43 mm to (147.5, 97.0), turned to -35 degrees
- moved D7 0.70 mm to (160.1, 94.5)
- moved D6 0.70 mm to (161.1, 94.5)
- moved D5 0.69 mm to (162.0, 94.5)
- moved C38 0.57 mm to (156.4, 92.0)
- moved R20 0.20 mm to (162.0, 95.4)
- moved R21 0.20 mm to (161.1, 95.4)
- moved R26 0.20 mm to (160.2, 95.4)
- moved C25 0.14 mm to (155.9, 93.9)
- moved R16 0.13 mm to (159.6, 96.9)
- moved C24 0.13 mm to (156.9, 93.9)
- moved C36 0.12 mm to (155.0, 93.9)
Routing:
- net GND: track 21.8 -> 26.0 mm, vias 22 -> 25
- net /GPS_RX: track 19.6 -> 17.5 mm
- net +3V3: track 18.1 -> 16.5 mm, vias 16 -> 18
- net /USB_DN: track 9.44 -> 11.0 mm
- net Net-(D7-A): track 0.88 -> 0.00 mm, vias 0 -> 1
- net Net-(D6-A): track 0.88 -> 0.00 mm, vias 0 -> 1
- net Net-(D5-A): track 0.88 -> 0.00 mm, vias 0 -> 1
- net /MCU/FLASH_CLK: track 8.04 -> 7.43 mm
- net /GPS_TX: track 18.7 -> 18.1 mm
- net /EN: track 28.9 -> 28.4 mm
- net /TX_RX: track 15.5 -> 15.0 mm
- net /LED_R: track 5.21 -> 5.11 mm, vias 0 -> 1
- net /LED_G: track 3.56 -> 3.62 mm, vias 0 -> 1
- net /LED_B: track 2.46 -> 2.52 mm, vias 0 -> 1
