File: fpv_drone/esc_ch1.kicad_sch (KiCad schematic)
At the start: 14 parts, among them J6 MOT1, Q2 IRFH5015, Q3 IRFH5015, Q4 IRFH5015, Q5 IRFH5015, Q6 IRFH5015, Q7 IRFH5015, U10 FD6288_ESC1, U9 STM32G071K_ESC1

Commit message: updated
Parts:
- removed Q2, Q3, Q4, Q5, Q6, Q7: IRFH5015, Package_TO_SOT_SMD:TO-263-2, symbol Transistor_FET:Q_NMOS_GDS
- added Q1, Q2, Q3, Q4, Q5, Q6: AON7418, AON7418:PDFN-8_L3.3-W3.3-P0.65-BL, symbol AON7418:AON7418
- renumbered C27 to C33, C28 to C34, C29 to C35, C30 to C36, C31 to C37, J6 to J7
Connections:
- net GND: now also Q2.1 (S), Q2.2 (S), Q2.3 (S), Q4.1 (S), Q4.2 (S), Q4.3 (S), Q6.1 (S), Q6.2 (S), Q6.3 (S)
- net HO1: now also Q1.4 (G)
- net HO2: now also Q3.4 (G)
- net HO3: now also Q5.4 (G)
- net LO1: now also Q2.4 (G)
- net LO2: now also Q4.4 (G)
- net LO3: now also Q6.4 (G)
- net VS1: now also Q1.1 (S), Q1.2 (S), Q1.3 (S), Q2.5 (D), Q2.6 (D), Q2.7 (D), Q2.8 (D), Q2.9 (D)
- net VS2: now also Q3.1 (S), Q3.2 (S), Q3.3 (S), Q4.5 (D), Q4.6 (D), Q4.7 (D), Q4.8 (D), Q4.9 (D)
- net VS3: now also Q5.1 (S), Q5.2 (S), Q5.3 (S), Q6.5 (D), Q6.6 (D), Q6.7 (D), Q6.8 (D), Q6.9 (D)
- net VBAT renamed +BATT
- net +BATT: now also Q1.5 (D), Q1.6 (D), Q1.7 (D), Q1.8 (D), Q1.9 (D), Q3.5 (D), Q3.6 (D), Q3.7 (D), Q3.8 (D), Q3.9 (D), Q5.5 (D), Q5.6 (D), Q5.7 (D), Q5.8 (D), Q5.9 (D)
Other:
- moved on the sheet: J7
