File: fpv_drone/esc_ch2.kicad_sch (KiCad schematic)
At the start: 14 parts, among them J8 MOT2, Q14 IRFH5015, Q15 IRFH5015, Q16 IRFH5015, Q17 IRFH5015, Q18 IRFH5015, Q19 IRFH5015, U13 STM32G071K_ESC2, U14 FD6288_ESC2

Commit message: updated
Parts:
- removed C39, C40, C41: 100nF, Capacitor_SMD:C_0603_1608Metric, symbol Device:C
- removed J8: MOT2, Connector_Wire:SolderWire-0.75sqmm_1x03_P7mm_D1.25mm_OD3.5mm, symbol Connector_Generic:Conn_01x03
- removed Q14, Q15, Q16, Q17, Q18, Q19: IRFH5015, Package_TO_SOT_SMD:TO-263-2, symbol Transistor_FET:Q_NMOS_GDS
- added C45, C46, C47: 100nF, Capacitor_SMD:C_0603_1608Metric, symbol Device:C
- added J9: MOT3, Connector_Wire:SolderWire-0.75sqmm_1x03_P7mm_D1.25mm_OD3.5mm, symbol Connector_Generic:Conn_01x03
- added Q13, Q14, Q15, Q16, Q17, Q18: AON7418, AON7418:PDFN-8_L3.3-W3.3-P0.65-BL, symbol AON7418:AON7418
- renumbered C37 to C43, C38 to C44
Connections:
- net GND: now also Q14.1 (S), Q14.2 (S), Q14.3 (S), Q16.1 (S), Q16.2 (S), Q16.3 (S), Q18.1 (S), Q18.2 (S), Q18.3 (S)
- net HO1: now also Q13.4 (G)
- net HO2: now also Q15.4 (G)
- net HO3: now also Q17.4 (G)
- net LO1: now also Q14.4 (G)
- net LO2: now also Q16.4 (G)
- net LO3: now also Q18.4 (G)
- net VB1: now also C45.1
- net VB2: now also C46.1
- net VB3: now also C47.1
- net VS1: now also C45.2, J9.1 (Pin_1), Q13.1 (S), Q13.2 (S), Q13.3 (S), Q14.5 (D), Q14.6 (D), Q14.7 (D), Q14.8 (D), Q14.9 (D)
- net VS2: now also C46.2, J9.2 (Pin_2), Q15.1 (S), Q15.2 (S), Q15.3 (S), Q16.5 (D), Q16.6 (D), Q16.7 (D), Q16.8 (D), Q16.9 (D)
- net VS3: now also C47.2, J9.3 (Pin_3), Q17.1 (S), Q17.2 (S), Q17.3 (S), Q18.5 (D), Q18.6 (D), Q18.7 (D), Q18.8 (D), Q18.9 (D)
- net VBAT renamed +BATT
- net +BATT: now also Q13.5 (D), Q13.6 (D), Q13.7 (D), Q13.8 (D), Q13.9 (D), Q15.5 (D), Q15.6 (D), Q15.7 (D), Q15.8 (D), Q15.9 (D), Q17.5 (D), Q17.6 (D), Q17.7 (D), Q17.8 (D), Q17.9 (D)
