File: fpv_drone/esc_ch3.kicad_sch (KiCad schematic)
At the start: 14 parts, among them J7 MOT3, Q10 IRFH5015, Q11 IRFH5015, Q12 IRFH5015, Q13 IRFH5015, Q8 IRFH5015, Q9 IRFH5015, U11 STM32G071K_ESC3, U12 FD6288_ESC3

Commit message: updated
Parts:
- removed Q10, Q11, Q12, Q13, Q8, Q9: IRFH5015, Package_TO_SOT_SMD:TO-263-2, symbol Transistor_FET:Q_NMOS_GDS
- added Q10, Q11, Q12, Q7, Q8, Q9: AON7418, AON7418:PDFN-8_L3.3-W3.3-P0.65-BL, symbol AON7418:AON7418
- renumbered C32 to C38, C33 to C39, C34 to C40, C35 to C41, C36 to C42, J7 to J8
Connections:
- net GND: now also Q10.1 (S), Q10.2 (S), Q10.3 (S), Q12.1 (S), Q12.2 (S), Q12.3 (S), Q8.1 (S), Q8.2 (S), Q8.3 (S)
- net HO1: now also Q7.4 (G)
- net HO2: now also Q9.4 (G)
- net HO3: now also Q11.4 (G)
- net LO1: now also Q8.4 (G)
- net LO2: now also Q10.4 (G)
- net LO3: now also Q12.4 (G)
- net VS1: now also Q7.1 (S), Q7.2 (S), Q7.3 (S), Q8.5 (D), Q8.6 (D), Q8.7 (D), Q8.8 (D), Q8.9 (D)
- net VS2: now also Q10.5 (D), Q10.6 (D), Q10.7 (D), Q10.8 (D), Q10.9 (D), Q9.1 (S), Q9.2 (S), Q9.3 (S)
- net VS3: now also Q11.1 (S), Q11.2 (S), Q11.3 (S), Q12.5 (D), Q12.6 (D), Q12.7 (D), Q12.8 (D), Q12.9 (D)
- net VBAT renamed +BATT
- net +BATT: now also Q11.5 (D), Q11.6 (D), Q11.7 (D), Q11.8 (D), Q11.9 (D), Q7.5 (D), Q7.6 (D), Q7.7 (D), Q7.8 (D), Q7.9 (D), Q9.5 (D), Q9.6 (D), Q9.7 (D), Q9.8 (D), Q9.9 (D)
Other:
- moved on the sheet: J8
