File: fpv_drone/esc_ch4.kicad_sch (KiCad schematic)
At the start: 14 parts, among them J9 MOT4, Q20 IRFH5015, Q21 IRFH5015, Q22 IRFH5015, Q23 IRFH5015, Q24 IRFH5015, Q25 IRFH5015, U15 STM32G071K_ESC4, U16 FD6288_ESC4

Commit message: updated
Parts:
- removed C44, C45, C46: 100nF, Capacitor_SMD:C_0603_1608Metric, symbol Device:C
- removed J9: MOT4, Connector_Wire:SolderWire-0.75sqmm_1x03_P7mm_D1.25mm_OD3.5mm, symbol Connector_Generic:Conn_01x03
- removed Q20, Q21, Q22, Q23, Q24, Q25: IRFH5015, Package_TO_SOT_SMD:TO-263-2, symbol Transistor_FET:Q_NMOS_GDS
- added C50, C51, C52: 100nF, Capacitor_SMD:C_0603_1608Metric, symbol Device:C
- added J10: MOT3, Connector_Wire:SolderWire-0.75sqmm_1x03_P7mm_D1.25mm_OD3.5mm, symbol Connector_Generic:Conn_01x03
- added Q19, Q20, Q21, Q22, Q23, Q24: AON7418, AON7418:PDFN-8_L3.3-W3.3-P0.65-BL, symbol AON7418:AON7418
- renumbered C42 to C48, C43 to C49
Connections:
- net GND: now also Q20.1 (S), Q20.2 (S), Q20.3 (S), Q22.1 (S), Q22.2 (S), Q22.3 (S), Q24.1 (S), Q24.2 (S), Q24.3 (S)
- net HO1: now also Q19.4 (G)
- net HO2: now also Q21.4 (G)
- net HO3: now also Q23.4 (G)
- net LO1: now also Q20.4 (G)
- net LO2: now also Q22.4 (G)
- net LO3: now also Q24.4 (G)
- net VB1: now also C50.1
- net VB2: now also C51.1
- net VB3: now also C52.1
- net VS1: now also C50.2, J10.1 (Pin_1), Q19.1 (S), Q19.2 (S), Q19.3 (S), Q20.5 (D), Q20.6 (D), Q20.7 (D), Q20.8 (D), Q20.9 (D)
- net VS2: now also C51.2, J10.2 (Pin_2), Q21.1 (S), Q21.2 (S), Q21.3 (S), Q22.5 (D), Q22.6 (D), Q22.7 (D), Q22.8 (D), Q22.9 (D)
- net VS3: now also C52.2, J10.3 (Pin_3), Q23.1 (S), Q23.2 (S), Q23.3 (S), Q24.5 (D), Q24.6 (D), Q24.7 (D), Q24.8 (D), Q24.9 (D)
- net VBAT renamed +BATT
- net +BATT: now also Q19.5 (D), Q19.6 (D), Q19.7 (D), Q19.8 (D), Q19.9 (D), Q21.5 (D), Q21.6 (D), Q21.7 (D), Q21.8 (D), Q21.9 (D), Q23.5 (D), Q23.6 (D), Q23.7 (D), Q23.8 (D), Q23.9 (D)
