File: fpv_drone/flight_controller.kicad_sch (KiCad schematic)
At the start: 15 parts, among them J5 USB-C, U8 STM32F405RGTx, Y3 8MHz

Commit message: updated
Parts:
- added C10: 1µF, Capacitor_SMD:C_0402_1005Metric, symbol Device:C
- added C5, C6, C7: 100nF, Capacitor_SMD:C_0402_1005Metric, symbol Device:C
- renumbered C20 to C26, C21 to C27, C22 to C28, C23 to C29, C24 to C30, C25 to C31, C26 to C32, J5 to J6, R7 to R10, R8 to R11, R9 to R12, R10 to R13, R11 to R14, Y3 to Y4
Connections:
- net +3V3: now also C10.2, C5.2, C6.2, C7.2
- net GND: now also C10.1, C5.1, C6.1, C7.1
- net IMU_ACC_CS: now reaches U8.10 (PC2)
- no-connect marks 25 -> 24
Other:
- moved on the sheet: C31, C32
