File: fpv_drone/fpv_drone.kicad_pcb (KiCad board)
At the start: 2 copper layers, 0 parts

Commit message: updated
Parts:
- added ?: , , F.Cu at (150.0, 140.1)
- added ?: , , F.Cu at (200.2, 132.8)
- added ?: , , F.Cu at (226.1, 105.2)
- added ?: , , F.Cu at (245.7, 133.7)
- added ?: , , F.Cu at (220.0, 210.0)
- added ?: , , F.Cu at (226.1, 166.5)
- added ?: , , F.Cu at (255.3, 146.0)
- added ?: , , F.Cu at (220.0, 70.5)
- added ?: , , F.Cu at (211.5, 159.6)
- added ?: , , F.Cu at (290.0, 140.1)
- added C1: DNP, Capacitor_SMD:C_0402_1005Metric, B.Cu at (227.8, 157.3)
- added C10: 1µF, Capacitor_SMD:C_0402_1005Metric, F.Cu at (211.1, 131.7)
- added C11: 10µF, Capacitor_SMD:C_0805_2012Metric, B.Cu at (225.0, 131.3)
- added C12: 22µF, Capacitor_SMD:C_0805_2012Metric, B.Cu at (235.8, 130.4)
- added C13: 100nF, Capacitor_SMD:C_0402_1005Metric, B.Cu at (224.0, 162.6)
- added C14: 100nF, Capacitor_SMD:C_0402_1005Metric, B.Cu at (224.2, 156.2)
- added C15: 100nF, Capacitor_SMD:C_0402_1005Metric, B.Cu at (228.7, 162.5)
- added C16: 10pF, Capacitor_SMD:C_0402_1005Metric, B.Cu at (216.9, 145.8)
- added C17: 10pF, Capacitor_SMD:C_0402_1005Metric, B.Cu at (218.7, 145.8)
- added C18: 1µF, Capacitor_SMD:C_0402_1005Metric, B.Cu at (222.6, 147.3)
- added C19: 100nF, Capacitor_SMD:C_0402_1005Metric, B.Cu at (224.0, 153.7)
- added C2: 470µF/25V, Capacitor_SMD:C_Elec_6.3x5.8, F.Cu at (216.8, 124.0)
- added C20: 100nF, Capacitor_SMD:C_0402_1005Metric, B.Cu at (224.0, 150.8)
- added C21: 100nF, Capacitor_SMD:C_0402_1005Metric, B.Cu at (219.8, 147.3)
- added C22: 100nF, Capacitor_SMD:C_0402_1005Metric, B.Cu at (217.3, 158.9)
- added C23: 100nF, Capacitor_SMD:C_0402_1005Metric, F.Cu at (233.4, 133.2)
- added C24: 100nF, Capacitor_SMD:C_0402_1005Metric, F.Cu at (231.0, 130.0)
- added C25: 100nF, Capacitor_SMD:C_0402_1005Metric, F.Cu at (221.9, 136.8)
- added C26: 20pF, Capacitor_SMD:C_0402_1005Metric, F.Cu at (218.8, 129.1)
- added C27: 20pF, Capacitor_SMD:C_0402_1005Metric, F.Cu at (214.4, 131.7)
- added C28: 100nF, Capacitor_SMD:C_0402_1005Metric, F.Cu at (213.5, 131.6)
- added C29: 2.2µF, Capacitor_SMD:C_0603_1608Metric, F.Cu at (203.7, 145.1)
- added C3: 10µF, Capacitor_SMD:C_0805_2012Metric, B.Cu at (222.8, 124.4)
- added C30: 2.2µF, Capacitor_SMD:C_0603_1608Metric, F.Cu at (219.0, 147.9)
- added C31: 100nF, Capacitor_SMD:C_0402_1005Metric, F.Cu at (204.3, 146.4)
- added C32: 100nF, Capacitor_SMD:C_0402_1005Metric, F.Cu at (210.2, 131.7)
- added C33: 100nF, Capacitor_SMD:C_0402_1005Metric, F.Cu at (227.0, 110.9)
- added C34: 100nF, Capacitor_SMD:C_0402_1005Metric, B.Cu at (214.9, 110.2)
- added C35: 100nF, Capacitor_SMD:C_0603_1608Metric, F.Cu at (219.3, 98.9)
- added C36: 100nF, Capacitor_SMD:C_0603_1608Metric, F.Cu at (219.3, 91.9)
- added C37: 100nF, Capacitor_SMD:C_0603_1608Metric, F.Cu at (219.3, 84.9)
- added C38: 100nF, Capacitor_SMD:C_0402_1005Metric, F.Cu at (213.5, 169.2)
- added C39: 100nF, Capacitor_SMD:C_0402_1005Metric, B.Cu at (225.3, 170.0)
- added C4: 100nF, Capacitor_SMD:C_0402_1005Metric, B.Cu at (219.1, 121.3)
- added C40: 100nF, Capacitor_SMD:C_0603_1608Metric, F.Cu at (220.7, 181.6)
- added C41: 100nF, Capacitor_SMD:C_0603_1608Metric, F.Cu at (220.7, 188.6)
- added C42: 100nF, Capacitor_SMD:C_0603_1608Metric, F.Cu at (220.7, 195.6)
- added C43: 100nF, Capacitor_SMD:C_0402_1005Metric, F.Cu at (190.3, 133.6)
- added C44: 100nF, Capacitor_SMD:C_0402_1005Metric, B.Cu at (189.4, 145.7)
- added C45: 100nF, Capacitor_SMD:C_0603_1608Metric, F.Cu at (178.0, 140.8)
- added C46: 100nF, Capacitor_SMD:C_0603_1608Metric, F.Cu at (171.0, 140.8)
- added C47: 100nF, Capacitor_SMD:C_0603_1608Metric, F.Cu at (164.0, 140.8)
- added C48: 100nF, Capacitor_SMD:C_0402_1005Metric, F.Cu at (250.0, 146.3)
- added C49: 100nF, Capacitor_SMD:C_0402_1005Metric, B.Cu at (250.5, 134.8)
- added C5: 100nF, Capacitor_SMD:C_0402_1005Metric, F.Cu at (218.7, 134.7)
- added C50: 100nF, Capacitor_SMD:C_0603_1608Metric, F.Cu at (261.8, 139.0)
- added C51: 100nF, Capacitor_SMD:C_0603_1608Metric, F.Cu at (268.8, 139.0)
- added C52: 100nF, Capacitor_SMD:C_0603_1608Metric, F.Cu at (275.8, 139.0)
- added C53: 100nF, Capacitor_SMD:C_0402_1005Metric, F.Cu at (200.2, 142.3)
- added C54: 100nF, Capacitor_SMD:C_0402_1005Metric, F.Cu at (204.2, 138.6)
- added C55: 100nF, Capacitor_SMD:C_0402_1005Metric, F.Cu at (238.0, 139.1)
- added C56: 100nF, Capacitor_SMD:C_0402_1005Metric, F.Cu at (233.9, 139.1)
- added C57: 100nF, Capacitor_SMD:C_0402_1005Metric, F.Cu at (231.1, 143.3)
- added C58: 10µF, Capacitor_SMD:C_0805_2012Metric, B.Cu at (224.4, 152.2)
- added C59: 100nF, Capacitor_SMD:C_0402_1005Metric, B.Cu at (220.7, 147.3)
- added C6: 100nF, Capacitor_SMD:C_0402_1005Metric, F.Cu at (218.4, 146.7)
- added C60: DNP, Capacitor_SMD:C_0402_1005Metric, B.Cu at (228.5, 156.7)
- added C7: 100nF, Capacitor_SMD:C_0402_1005Metric, F.Cu at (219.7, 134.7)
- added C8: 100nF, Capacitor_SMD:C_0402_1005Metric, B.Cu at (221.7, 118.2)
- added C9: 22µF, Capacitor_SMD:C_0805_2012Metric, B.Cu at (222.1, 127.1)
- added D2: SMBJ20A, Diode_SMD:D_SMA, B.Cu at (216.8, 124.0)
- added D3: WS2812B, LED_SMD:LED_WS2812B_PLCC4_5.0x5.0mm_P3.2mm, F.Cu at (214.1, 115.6)
- added G***: LOGO, LOGO, F.Cu at (234.3, 150.9)
- added J10: MOT3, Connector_Wire:SolderWire-0.75sqmm_1x03_P7mm_D1.25mm_OD3.5mm, F.Cu at (263.8, 135.3)
- added J11: BUZZER, Buzzer_Beeper:MagneticBuzzer_Kobitone_254-EMB84Q-RO, F.Cu at (218.4, 153.7)
- added J12: SWD_DEBUG, Connector_PinHeader_1.27mm:PinHeader_1x04_P1.27mm_Vertical, F.Cu at (224.6, 148.9)
- added J2: BATT, Connector_AMASS:AMASS_XT30UPB-M_1x02_P5.0mm_Vertical, F.Cu at (205.0, 130.4)
- added J4: CAM, Connector_JST:JST_SH_SM03B-SRSS-TB_1x03-1MP_P1.00mm_Horizontal, F.Cu at (239.8, 132.1)
- added J5: VTX_MODULE, Connector_JST:JST_SH_SM06B-SRSS-TB_1x06-1MP_P1.00mm_Horizontal, F.Cu at (231.0, 125.2)
- added J6: USB-C, Connector_USB:USB_C_Receptacle_GCT_USB4085, B.Cu at (211.6, 152.6)
- added J7: MOT1, Connector_Wire:SolderWire-0.75sqmm_1x03_P7mm_D1.25mm_OD3.5mm, F.Cu at (215.5, 96.8)
- added J8: MOT3, Connector_Wire:SolderWire-0.75sqmm_1x03_P7mm_D1.25mm_OD3.5mm, F.Cu at (224.4, 183.6)
- added J9: MOT3, Connector_Wire:SolderWire-0.75sqmm_1x03_P7mm_D1.25mm_OD3.5mm, F.Cu at (175.9, 144.5)
- added L1: 1.5nH, Inductor_SMD:L_0402_1005Metric, B.Cu at (229.2, 158.0)
- added L2: 4.7µH, Inductor_SMD:L_6.3x6.3_H3, B.Cu at (227.2, 123.5)
- added Q1: AON7418, AON7418:PDFN-8_L3.3-W3.3-P0.65-BL, B.Cu at (219.9, 96.2)
- added Q10: AON7418, AON7418:PDFN-8_L3.3-W3.3-P0.65-BL, F.Cu at (220.1, 191.3)
- added Q11: AON7418, AON7418:PDFN-8_L3.3-W3.3-P0.65-BL, B.Cu at (220.1, 198.2)
- added Q12: AON7418, AON7418:PDFN-8_L3.3-W3.3-P0.65-BL, F.Cu at (220.1, 198.2)
- added Q13: AON7418, AON7418:PDFN-8_L3.3-W3.3-P0.65-BL, B.Cu at (175.3, 140.1)
- added Q14: AON7418, AON7418:PDFN-8_L3.3-W3.3-P0.65-BL, F.Cu at (175.3, 140.1)
- added Q15: AON7418, AON7418:PDFN-8_L3.3-W3.3-P0.65-BL, B.Cu at (168.3, 140.1)
- added Q16: AON7418, AON7418:PDFN-8_L3.3-W3.3-P0.65-BL, F.Cu at (168.3, 140.1)
- added Q17: AON7418, AON7418:PDFN-8_L3.3-W3.3-P0.65-BL, B.Cu at (161.3, 140.1)
- added Q18: AON7418, AON7418:PDFN-8_L3.3-W3.3-P0.65-BL, F.Cu at (161.3, 140.1)
- added Q19: AON7418, AON7418:PDFN-8_L3.3-W3.3-P0.65-BL, B.Cu at (264.5, 139.6)
- added Q2: AON7418, AON7418:PDFN-8_L3.3-W3.3-P0.65-BL, F.Cu at (219.9, 96.2)
- added Q20: AON7418, AON7418:PDFN-8_L3.3-W3.3-P0.65-BL, F.Cu at (264.5, 139.6)
- added Q21: AON7418, AON7418:PDFN-8_L3.3-W3.3-P0.65-BL, B.Cu at (271.5, 139.6)
- added Q22: AON7418, AON7418:PDFN-8_L3.3-W3.3-P0.65-BL, F.Cu at (271.5, 139.6)
- added Q23: AON7418, AON7418:PDFN-8_L3.3-W3.3-P0.65-BL, B.Cu at (278.4, 139.6)
- added Q24: AON7418, AON7418:PDFN-8_L3.3-W3.3-P0.65-BL, F.Cu at (278.4, 139.6)
- added Q26: BSS138, Package_TO_SOT_SMD:SOT-23, F.Cu at (222.0, 131.3)
- added Q3: AON7418, AON7418:PDFN-8_L3.3-W3.3-P0.65-BL, B.Cu at (219.9, 89.2)
- added Q4: AON7418, AON7418:PDFN-8_L3.3-W3.3-P0.65-BL, F.Cu at (219.9, 89.2)
- added Q5: AON7418, AON7418:PDFN-8_L3.3-W3.3-P0.65-BL, B.Cu at (219.9, 82.2)
- added Q6: AON7418, AON7418:PDFN-8_L3.3-W3.3-P0.65-BL, F.Cu at (219.9, 82.2)
- added Q7: AON7418, AON7418:PDFN-8_L3.3-W3.3-P0.65-BL, B.Cu at (220.1, 184.2)
- added Q8: AON7418, AON7418:PDFN-8_L3.3-W3.3-P0.65-BL, F.Cu at (220.1, 184.2)
- added Q9: AON7418, AON7418:PDFN-8_L3.3-W3.3-P0.65-BL, B.Cu at (220.1, 191.3)
- added R10: 10k, Resistor_SMD:R_0402_1005Metric, F.Cu at (222.5, 139.6)
- added R11: 5.1k, Resistor_SMD:R_0402_1005Metric, F.Cu at (211.6, 151.4)
- added R12: 5.1k, Resistor_SMD:R_0402_1005Metric, F.Cu at (206.4, 150.6)
- added R13: 22, Resistor_SMD:R_0402_1005Metric, F.Cu at (210.2, 149.1)
- added R14: 22, Resistor_SMD:R_0402_1005Metric, F.Cu at (210.8, 149.8)
- added R15: 100k, Resistor_SMD:R_0402_1005Metric, F.Cu at (222.8, 124.0)
- added R16: 100k, Resistor_SMD:R_0402_1005Metric, F.Cu at (221.1, 124.5)
- added R17: 4.7k, Resistor_SMD:R_0402_1005Metric, F.Cu at (238.5, 141.4)
- added R18: 4.7k, Resistor_SMD:R_0402_1005Metric, F.Cu at (238.5, 140.5)
- added R2: 73.2k, Resistor_SMD:R_0402_1005Metric, B.Cu at (220.1, 123.2)
- added R3: 10k, Resistor_SMD:R_0402_1005Metric, B.Cu at (221.1, 123.5)
- added R6: 12k, Resistor_SMD:R_0402_1005Metric, B.Cu at (221.6, 147.3)
- added R7: 10k, Resistor_SMD:R_0402_1005Metric, B.Cu at (223.5, 149.3)
- added R8: 10k, Resistor_SMD:R_0402_1005Metric, B.Cu at (224.0, 154.6)
- added R9: 10k, Resistor_SMD:R_0402_1005Metric, B.Cu at (217.8, 157.5)
- added REF**: MountingHole_2.2mm_M2_DIN965_Pad, MountingHole:MountingHole_2.2mm_M2_DIN965_Pad, F.Cu at (200.2, 148.4)
- added U10: FD6288_ESC1, FD6288T:TSSOP-20_L6.5-W4.4-P0.65-LS6.4-BL, B.Cu at (216.2, 105.2)
- added U11: STM32G071K_ESC3, Package_QFP:LQFP-32_7x7mm_P0.8mm, F.Cu at (217.6, 165.2)
- added U12: FD6288_ESC3, FD6288T:TSSOP-20_L6.5-W4.4-P0.65-LS6.4-BL, B.Cu at (224.0, 175.0)
- added U13: STM32G071K_ESC2, Package_QFP:LQFP-32_7x7mm_P0.8mm, F.Cu at (194.5, 137.8)
- added U14: FD6288_ESC2, FD6288T:TSSOP-20_L6.5-W4.4-P0.65-LS6.4-BL, B.Cu at (184.5, 144.4)
- added U15: STM32G071K_ESC4, Package_QFP:LQFP-32_7x7mm_P0.8mm, F.Cu at (245.7, 142.0)
- added U16: FD6288_ESC4, FD6288T:TSSOP-20_L6.5-W4.4-P0.65-LS6.4-BL, B.Cu at (255.3, 136.1)
- added U17: BMI088, Package_LGA:Bosch_LGA-16_4.5x3mm_P0.5mm_LayoutBorder7x1y_ClockwisePinNumbering, F.Cu at (203.3, 141.8)
- added U18: BMP280, Package_LGA:Bosch_LGA-8_2x2.5mm_P0.65mm_ClockwisePinNumbering, F.Cu at (235.9, 140.1)
- added U19: W25Q128JVS, Package_SO:SOIC-8_5.3x5.3mm_P1.27mm, F.Cu at (226.0, 144.4)
- added U2: TPS54302_5V, Package_TO_SOT_SMD:SOT-23-6, B.Cu at (221.7, 120.8)
- added U4: AMS1117-3.3, Package_TO_SOT_SMD:SOT-223-3_TabPin2, B.Cu at (230.4, 131.4)
- added U5: SX1280, SX1280IMLTRT:QFN-24_L4.0-W4.0-P0.50-BL-EP2.6, B.Cu at (226.5, 160.3)
- added U6: ESP8266EX, Package_DFN_QFN:QFN-32-1EP_5x5mm_P0.5mm_EP3.45x3.45mm, B.Cu at (218.7, 152.6)
- added U7: AT7456E, AT7456E:TSSOP-28_L9.7-W4.4-P0.65-LS6.4-BL-EP-2, F.Cu at (228.7, 135.4)
- added U8: STM32F405RGTx, Package_QFP:LQFP-64_10x10mm_P0.5mm, F.Cu at (213.4, 141.0)
- added U9: STM32G071K_ESC1, Package_QFP:LQFP-32_7x7mm_P0.8mm, F.Cu at (222.9, 114.9)
- added Y2: 26MHz, Crystal:Crystal_SMD_2012-2Pin_2.0x1.2mm, B.Cu at (217.8, 147.3)
- added Y3: 27MHz, Crystal:Crystal_SMD_3215-2Pin_3.2x1.5mm, F.Cu at (223.6, 138.5)
- added Y4: 8MHz, Crystal:Crystal_SMD_3225-4Pin_3.2x2.5mm, F.Cu at (217.1, 131.3)
Routing:
- net +BATT: track 0.00 -> 123.7 mm, vias 0 -> 18
- net /ESC_RX: track 0.00 -> 108.8 mm, vias 0 -> 7
- net +3V3: track 0.00 -> 97.4 mm, vias 0 -> 23
- net GND: track 0.00 -> 89.7 mm, vias 0 -> 39
- net /ESC/Motor 2/HO3: track 0.00 -> 41.2 mm
- net /ESC/Motor 1/HO3: track 0.00 -> 40.5 mm
- net /ESC/Motor 4/HO3: track 0.00 -> 39.7 mm, vias 0 -> 1
- net /ESC/Motor 3/HO3: track 0.00 -> 39.4 mm
- net /MOT4_PWM: track 0.00 -> 36.9 mm, vias 0 -> 2
- net /ESC/Motor 1/LO3: track 0.00 -> 36.7 mm, vias 0 -> 2
- net /ESC/Motor 2/LO3: track 0.00 -> 36.4 mm, vias 0 -> 2
- net /ESC/Motor 3/LO3: track 0.00 -> 36.4 mm, vias 0 -> 2
- net /ESC/Motor 4/LO3: track 0.00 -> 36.1 mm, vias 0 -> 2
- net /ESC/Motor 1/VB3: track 0.00 -> 31.7 mm, vias 0 -> 1
- net /MOT1_PWM: track 0.00 -> 30.6 mm, vias 0 -> 2
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- added copper zone on B.Cu, net +3V3
- added copper zone on In4.Cu, net +3V3
- added copper zone on B.Cu, net +5V
- added copper zone on In4.Cu, net +5V
- added copper zone on B.Cu, net +BATT
- added copper zone on B.Cu, net /ESC/Motor 1/VS1
- added copper zone on F.Cu, net /ESC/Motor 1/VS1
- added copper zone on B.Cu, net /ESC/Motor 1/VS2
- added copper zone on F.Cu, net /ESC/Motor 1/VS2
- added copper zone on B.Cu, net /ESC/Motor 1/VS3
- added copper zone on F.Cu, net /ESC/Motor 1/VS3
- added copper zone on B.Cu, net /ESC/Motor 2/VS1
- added copper zone on F.Cu, net /ESC/Motor 2/VS1
- added copper zone on B.Cu, net /ESC/Motor 2/VS2
- added copper zone on F.Cu, net /ESC/Motor 2/VS2
- added copper zone on B.Cu, net /ESC/Motor 2/VS3
- added copper zone on F.Cu, net /ESC/Motor 2/VS3
- added copper zone on B.Cu, net /ESC/Motor 3/VS1
- added copper zone on F.Cu, net /ESC/Motor 3/VS1
- added copper zone on B.Cu, net /ESC/Motor 3/VS2
- added copper zone on F.Cu, net /ESC/Motor 3/VS2
- added copper zone on B.Cu, net /ESC/Motor 3/VS3
- added copper zone on F.Cu, net /ESC/Motor 3/VS3
- added copper zone on B.Cu, net /ESC/Motor 4/VS1
- added copper zone on F.Cu, net /ESC/Motor 4/VS1
- added copper zone on B.Cu, net /ESC/Motor 4/VS2
- added copper zone on F.Cu, net /ESC/Motor 4/VS2
- added copper zone on B.Cu, net /ESC/Motor 4/VS3
- added copper zone on F.Cu, net /ESC/Motor 4/VS3
- added copper zone on B.Cu, net /Power Supply/FB_5V
- added copper zone on B.Cu, net GND
- added copper zone on F.Cu, net GND
- added copper zone on In1.Cu, net GND
- added copper zone on In2.Cu, net GND
- added copper zone on In3.Cu, net GND
Other:
- board outline added: 158 x 158 mm
- copper layers 2 -> 6
- rule pad_to_mask_clearance: 0 -> 0.051
