File: fpv_drone/fpv_drone.kicad_pcb (KiCad board)
At the start: 6 copper layers, 158 x 158 mm, 146 parts, among them J10 MOT3, J11 BUZZER, J12 SWD_DEBUG, J2 BATT, J4 CAM, J5 VTX_MODULE, J6 USB-C, J7 MOT1, J8 MOT3, J9 MOT3, Q1 AON7418, Q10 AON7418, Q11 AON7418, Q12 AON7418, Q13 AON7418, Q14 AON7418, Q15 AON7418, Q16 AON7418, Q17 AON7418, Q18 AON7418, Q19 AON7418, Q2 AON7418, Q20 AON7418, Q21 AON7418, Q22 AON7418, Q23 AON7418, Q24 AON7418, Q26 BSS138, Q3 AON7418, Q4 AON7418, Q5 AON7418, Q6 AON7418, Q7 AON7418, Q8 AON7418, Q9 AON7418, U10 FD6288_ESC1, U11 STM32G071K_ESC3, U12 FD6288_ESC3, U13 STM32G071K_ESC2, U14 FD6288_ESC2, U15 STM32G071K_ESC4, U16 FD6288_ESC4, U17 BMI088, U18 BMP280, U19 W25Q128JVS, U2 TPS54302_5V, U4 AMS1117-3.3, U5 SX1280, U6 ESP8266EX, U7 AT7456E, U8 STM32F405RGTx, U9 STM32G071K_ESC1, Y2 26MHz, Y3 27MHz, Y4 8MHz

Commit message: holes
Parts:
- removed the ? at (150.0, 140.1)
- removed the ? at (220.0, 210.0)
- removed the ? at (220.0, 70.5)
- removed the ? at (290.0, 140.1)
- added REF**: MountingHole_3.2mm_M3_DIN965_Pad, MountingHole:MountingHole_3.2mm_M3_DIN965_Pad, F.Cu at (214.1, 64.4)
- added REF**: MountingHole_3.2mm_M3_DIN965_Pad, MountingHole:MountingHole_3.2mm_M3_DIN965_Pad, F.Cu at (225.5, 64.7)
- added REF**: MountingHole_3.2mm_M3_DIN965_Pad, MountingHole:MountingHole_3.2mm_M3_DIN965_Pad, F.Cu at (214.3, 215.7)
- added REF**: MountingHole_3.2mm_M3_DIN965_Pad, MountingHole:MountingHole_3.2mm_M3_DIN965_Pad, F.Cu at (296.0, 134.1)
- added REF**: MountingHole_3.2mm_M3_DIN965_Pad, MountingHole:MountingHole_3.2mm_M3_DIN965_Pad, F.Cu at (284.3, 134.4)
- added REF**: MountingHole_3.2mm_M3_DIN965_Pad, MountingHole:MountingHole_3.2mm_M3_DIN965_Pad, F.Cu at (225.8, 76.7)
- added REF**: MountingHole_3.2mm_M3_DIN965_Pad, MountingHole:MountingHole_3.2mm_M3_DIN965_Pad, F.Cu at (155.7, 145.7)
- added REF**: MountingHole_3.2mm_M3_DIN965_Pad, MountingHole:MountingHole_3.2mm_M3_DIN965_Pad, F.Cu at (225.6, 204.4)
- added REF**: MountingHole_3.2mm_M3_DIN965_Pad, MountingHole:MountingHole_3.2mm_M3_DIN965_Pad, F.Cu at (214.0, 204.0)
- added REF**: MountingHole_3.2mm_M3_DIN965_Pad, MountingHole:MountingHole_3.2mm_M3_DIN965_Pad, F.Cu at (214.5, 76.3)
- added REF**: MountingHole_3.2mm_M3_DIN965_Pad, MountingHole:MountingHole_3.2mm_M3_DIN965_Pad, F.Cu at (156.0, 134.0)
- added REF**: MountingHole_3.2mm_M3_DIN965_Pad, MountingHole:MountingHole_3.2mm_M3_DIN965_Pad, F.Cu at (226.0, 216.1)
- added REF**: MountingHole_3.2mm_M3_DIN965_Pad, MountingHole:MountingHole_3.2mm_M3_DIN965_Pad, F.Cu at (144.3, 134.4)
- added REF**: MountingHole_3.2mm_M3_DIN965_Pad, MountingHole:MountingHole_3.2mm_M3_DIN965_Pad, F.Cu at (144.0, 146.1)
- added REF**: MountingHole_3.2mm_M3_DIN965_Pad, MountingHole:MountingHole_3.2mm_M3_DIN965_Pad, F.Cu at (295.6, 145.7)
- added REF**: MountingHole_3.2mm_M3_DIN965_Pad, MountingHole:MountingHole_3.2mm_M3_DIN965_Pad, F.Cu at (284.0, 146.1)
