File: fpv_drone/fpv_drone.kicad_sch (KiCad schematic)
At the start: 0 parts

Commit message: updated
Other:
- sheet Flight Controller ports: added IMU_ACC_CS; removed none
- sheet IMU and Sensors ports: added IMU_ACC_CS; removed none
Changed lines of the file:
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@@
 	(generator_version "10.0")
 	(paper "A4")
+	(wire
+		(pts
+			(xy 147.32 130.81) (xy 152.4 130.81)
+		)
+		(stroke
+			(width 0)
+			(type default)
+		)
+	)
 	(label "SPI2_MOSI"
 		(at 147.32 127 180)
@@
 		)
 	)
+	(label "IMU_ACC_CS"
+		(at 88.9 96.52 180)
+		(effects
+			(font
+				(size 1.27 1.27)
+				(line_spacing 0)
+			)
+			(justify right bottom)
+		)
+	)
 	(label "IMU_CS"
 		(at 88.9 78.74 180)
@@
 	(label "SWDIO"
 		(at 147.32 82.55 180)
+		(effects
+			(font
+				(size 1.27 1.27)
+				(line_spacing 0)
+			)
+			(justify right bottom)
+		)
+	)
+	(label "IMU_ACC_CS"
+		(at 147.32 130.81 180)
 		(effects
 			(font
@@
 			)
 		)
+		(pin "IMU_ACC_CS" input
+			(at 88.9 96.52 180)
+			(effects
+				(font
+					(size 1.27 1.27)
+				)
+				(justify left)
+			)
+		)
 	)
 	(sheet
@@
 			(effects
 				(font
+					(size 1.27 1.27)
+				)
+				(justify left)
+			)
+		)
+		(pin "IMU_ACC_CS" input
+			(at 147.32 130.81 180)
+			(effects
+				(font
