File: fpv_drone/imu_sensors.kicad_sch (KiCad schematic)
At the start: 12 parts, among them U2 ATmega32U4-A, Y1 16MHz

Commit message: new boards
Parts:
- removed C10, C11: 22pF, Capacitor_SMD:C_0402_1005Metric, symbol Device:C
- removed C2, C7, C8, C9: 100nF, Capacitor_SMD:C_0402_1005Metric, symbol Device:C
- removed C6: 1uF, Capacitor_SMD:C_0402_1005Metric, symbol Device:C
- removed R2, R9: 10k, Resistor_SMD:R_0402_1005Metric, symbol Device:R
- removed R6: 22, Resistor_SMD:R_0402_1005Metric, symbol Device:R
- removed U2: ATmega32U4-A, Package_QFP:TQFP-44_10x10mm_P0.8mm, symbol MCU_Microchip_ATmega:ATmega32U4-A
- removed Y1: 16MHz, Crystal:Crystal_SMD_HC49-SD, symbol Device:Crystal
- added C47, C48, C49, C50, C51: 100nF, Capacitor_SMD:C_0402_1005Metric, symbol Device:C
- added U17: BMI088, Package_LGA:Bosch_LGA-16_4.5x3mm_P0.5mm_LayoutBorder7x1y_ClockwisePinNumbering, symbol Sensor_Motion:BMI088
- added U18: BMP280, Package_LGA:Bosch_LGA-8_2x2.5mm_P0.65mm_ClockwisePinNumbering, symbol Sensor_Pressure:BMP280
- added U19: W25Q128JVS, Package_SO:SOIC-8_5.3x5.3mm_P1.27mm, symbol Memory_Flash:W25Q128JVS
Connections:
- net +3V3: now also C47.1, C48.2, C49.2, C50.2, C51.2, U17.11 (VDDIO), U17.3 (VDD), U18.2 (CSB), U18.6 (VDDIO), U18.8 (VDD), U19.3 (~{WP}/IO_{2}), U19.7 (~{HOLD}/~{RESET}/IO_{3}), U19.8 (VCC)
- net GND: now also C47.2, C48.1, C49.1, C50.1, C51.1, U17.2 (GNDA), U17.4 (GNDA), U17.6 (GNDIO), U17.7 (PS), U18.1 (GND), U18.5 (SDO), U18.7 (GND), U19.4 (GND)
- new net BARO_SCL: U18.4 (SCK)
- new net BARO_SDA: U18.3 (SDI)
- new net FLASH_CS: U19.1 (~{CS})
- new net IMU_CS: U17.14 (~{CSB1}), U17.5 (~{CSB2})
- new net IMU_MISO: U17.10 (SDO2), U17.15 (SDO1)
- new net IMU_MOSI: U17.9 (SDI/SDA)
- new net IMU_SCK: U17.8 (SCK/SCL)
- new net SPI2_MISO: U19.2 (DO/IO_{1})
- new net SPI2_MOSI: U19.5 (DI/IO_{0})
- new net SPI2_SCK: U19.6 (CLK)
- no-connect marks 14 -> 4

Commit message: updated
Parts:
- added R17, R18: 4.7k, Resistor_SMD:R_0402_1005Metric, symbol Device:R
- renumbered C47 to C53, C48 to C54, C49 to C55, C50 to C56, C51 to C57
Connections:
- net +3V3: now also R17.2, R18.2
- net BARO_SCL: now also R17.1
- net BARO_SDA: now also R18.1
- net IMU_CS: no longer U17.5 (~{CSB2})
- new net IMU_ACC_CS: U17.5 (~{CSB2})
