File: fpv_drone/osd_vtx.kicad_sch (KiCad schematic)
At the start: 7 parts, among them J3 CAM, J4 VTX_MODULE, U7 AT7456E, Y2 27MHz

Commit message: updated
Parts:
- J4: renamed from J3; footprint Connector_PinHeader_2.54mm:PinHeader_1x03_P2.54mm_Vertical -> Connector_JST:JST_SH_SM03B-SRSS-TB_1x03-1MP_P1.00mm_Horizontal
- J5: renamed from J4; footprint Connector_PinHeader_2.54mm:PinHeader_1x06_P2.54mm_Vertical -> Connector_JST:JST_SH_SM06B-SRSS-TB_1x06-1MP_P1.00mm_Horizontal
- renumbered C17 to C23, C18 to C24, C19 to C25, Y2 to Y3
Changed lines of the file:
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@@
 		(in_pos_files yes)
 		(dnp no)
-		(property "Reference" "#PWR038"
+		(property "Reference" "#PWR056"
 			(at 151.13 80.01 0)
 			(hide yes)
@@
 			(project ""
 				(path "/bcc951e4-6780-442e-8e93-0576bc471757/f7e313ad-53b3-434b-b9a9-dc814318d635"
-					(reference "#PWR038")
+					(reference "#PWR056")
 					(unit 1)
 				)
@@
 		(in_pos_files yes)
 		(dnp no)
-		(property "Reference" "Y2"
+		(property "Reference" "Y3"
 			(at 86.36 85.09 0)
 			(show_name no)
@@
 			(project ""
 				(path "/bcc951e4-6780-442e-8e93-0576bc471757/f7e313ad-53b3-434b-b9a9-dc814318d635"
-					(reference "Y2")
+					(reference "Y3")
 					(unit 1)
 				)
@@
 		(in_pos_files yes)
 		(dnp no)
-		(property "Reference" "#PWR034"
+		(property "Reference" "#PWR051"
 			(at 119.38 59.69 0)
 			(hide yes)
@@
 				)
 				(path "/bcc951e4-6780-442e-8e93-0576bc471757/f7e313ad-53b3-434b-b9a9-dc814318d635"
-					(reference "#PWR034")
+					(reference "#PWR051")
 					(unit 1)
 				)
@@
 		(in_pos_files yes)
 		(dnp no)
-		(property "Reference" "J3"
+		(property "Reference" "J4"
 			(at 209.55 69.85 0)
 			(show_name no)
@@
 			)
 		)
-		(property "Footprint" "Connector_PinHeader_2.54mm:PinHeader_1x03_P2.54mm_Vertical"
+		(property "Footprint" "Connector_JST:JST_SH_SM03B-SRSS-TB_1x03-1MP_P1.00mm_Horizontal"
 			(at 209.55 74.93 0)
 			(hide yes)
@@
 			)
 		)
+		(pin "2"
+		)
 		(pin "1"
 		)
 		(pin "3"
 		)
-		(pin "2"
-		)
-		(instances
-			(project ""
-				(path "/bcc951e4-6780-442e-8e93-0576bc471757/f7e313ad-53b3-434b-b9a9-dc814318d635"
-					(reference "J3")
+		(instances
+			(project "fpv_drone"
+				(path "/bcc951e4-6780-442e-8e93-0576bc471757/f7e313ad-53b3-434b-b9a9-dc814318d635"
+					(reference "J4")
 					(unit 1)
 				)
@@
 		(in_pos_files yes)
 		(dnp no)
-		(property "Reference" "C18"
+		(property "Reference" "C24"
 			(at 152.4 80.645 0)
 			(show_name no)
@@
 			(project ""
 				(path "/bcc951e4-6780-442e-8e93-0576bc471757/f7e313ad-53b3-434b-b9a9-dc814318d635"
-					(reference "C18")
+					(reference "C24")
 					(unit 1)
 				)
@@
 		(in_pos_files yes)
 		(dnp no)
-		(property "Reference" "#PWR033"
+		(property "Reference" "#PWR050"
 			(at 96.52 81.28 0)
 			(hide yes)
@@
 				)
 				(path "/bcc951e4-6780-442e-8e93-0576bc471757/f7e313ad-53b3-434b-b9a9-dc814318d635"
-					(reference "#PWR033")
+					(reference "#PWR050")
 					(unit 1)
 				)
@@
 		)
 		(property "Value" "AT7456E"
-			(at 119.38 90.17 0)
+			(at 119.38 87.122 0)
 			(show_name no)
 			(do_not_autoplace no)
@@
 		(in_pos_files yes)
 		(dnp no)
-		(property "Reference" "#PWR046"
+		(property "Reference" "#PWR064"
 			(at 203.2 99.06 0)
 			(hide yes)
@@
 			(project ""
 				(path "/bcc951e4-6780-442e-8e93-0576bc471757/f7e313ad-53b3-434b-b9a9-dc814318d635"
-					(reference "#PWR046")
+					(reference "#PWR064")
 					(unit 1)
 				)
@@
 		(in_pos_files yes)
 		(dnp no)
-		(property "Reference" "C19"
+		(property "Reference" "C25"
 			(at 157.48 92.075 0)
 			(show_name no)
@@
 			(project ""
 				(path "/bcc951e4-6780-442e-8e93-0576bc471757/f7e313ad-53b3-434b-b9a9-dc814318d635"
-					(reference "C19")
+					(reference "C25")
 					(unit 1)
 				)
@@
 		(in_pos_files yes)
 		(dnp no)
-		(property "Reference" "C17"
+		(property "Reference" "C23"
 			(at 102.235 62.23 0)
 			(show_name no)
@@
 			(project ""
 				(path "/bcc951e4-6780-442e-8e93-0576bc471757/f7e313ad-53b3-434b-b9a9-dc814318d635"
-					(reference "C17")
+					(reference "C23")
 					(unit 1)
 				)
@@
 		(in_pos_files yes)
 		(dnp no)
-		(property "Reference" "#PWR039"
+		(property "Reference" "#PWR057"
 			(at 166.37 81.28 0)
 			(hide yes)
@@
 			(project ""
 				(path "/bcc951e4-6780-442e-8e93-0576bc471757/f7e313ad-53b3-434b-b9a9-dc814318d635"
-					(reference "#PWR039")
+					(reference "#PWR057")
 					(unit 1)
 				)
@@
 		(in_pos_files yes)
 		(dnp no)
-		(property "Reference" "#PWR041"
+		(property "Reference" "#PWR059"
 			(at 193.04 106.68 0)
 			(hide yes)
@@
 			(project ""
 				(path "/bcc951e4-6780-442e-8e93-0576bc471757/f7e313ad-53b3-434b-b9a9-dc814318d635"
-					(reference "#PWR041")
+					(reference "#PWR059")
 					(unit 1)
 				)
@@
 		(in_pos_files yes)
 		(dnp no)
-		(property "Reference" "#PWR037"
+		(property "Reference" "#PWR054"
 			(at 144.78 100.33 0)
 			(hide yes)
@@
 				)
 				(path "/bcc951e4-6780-442e-8e93-0576bc471757/f7e313ad-53b3-434b-b9a9-dc814318d635"
-					(reference "#PWR037")
+					(reference "#PWR054")
 					(unit 1)
 				)
@@
 		(in_pos_files yes)
 		(dnp no)
-		(property "Reference" "#PWR040"
+		(property "Reference" "#PWR058"
 			(at 166.37 91.44 0)
 			(hide yes)
@@
 				)
 				(path "/bcc951e4-6780-442e-8e93-0576bc471757/f7e313ad-53b3-434b-b9a9-dc814318d635"
-					(reference "#PWR040")
+					(reference "#PWR058")
 					(unit 1)
 				)
@@
 		(in_pos_files yes)
 		(dnp no)
-		(property "Reference" "#PWR045"
+		(property "Reference" "#PWR063"
 			(at 203.2 76.2 0)
 			(hide yes)
@@
 			(project ""
 				(path "/bcc951e4-6780-442e-8e93-0576bc471757/f7e313ad-53b3-434b-b9a9-dc814318d635"
-					(reference "#PWR045")
+					(reference "#PWR063")
 					(unit 1)
 				)
@@
 		(in_pos_files yes)
 		(dnp no)
-		(property "Reference" "J4"
+		(property "Reference" "J5"
 			(at 209.55 92.71 0)
 			(show_name no)
@@
 			)
 		)
-		(property "Footprint" "Connector_PinHeader_2.54mm:PinHeader_1x06_P2.54mm_Vertical"
+		(property "Footprint" "Connector_JST:JST_SH_SM06B-SRSS-TB_1x06-1MP_P1.00mm_Horizontal"
 			(at 209.55 100.33 0)
 			(hide yes)
@@
 			)
 		)
+		(pin "1"
+		)
+		(pin "2"
+		)
 		(pin "3"
 		)
+		(pin "4"
+		)
 		(pin "5"
 		)
-		(pin "4"
-		)
-		(pin "1"
-		)
 		(pin "6"
 		)
-		(pin "2"
-		)
-		(instances
-			(project ""
-				(path "/bcc951e4-6780-442e-8e93-0576bc471757/f7e313ad-53b3-434b-b9a9-dc814318d635"
-					(reference "J4")
+		(instances
+			(project "fpv_drone"
+				(path "/bcc951e4-6780-442e-8e93-0576bc471757/f7e313ad-53b3-434b-b9a9-dc814318d635"
+					(reference "J5")
 					(unit 1)
 				)
@@
 		(in_pos_files yes)
 		(dnp no)
-		(property "Reference" "#PWR042"
+		(property "Reference" "#PWR060"
 			(at 199.39 101.6 0)
 			(hide yes)
@@
 			(project ""
 				(path "/bcc951e4-6780-442e-8e93-0576bc471757/f7e313ad-53b3-434b-b9a9-dc814318d635"
-					(reference "#PWR042")
+					(reference "#PWR060")
 					(unit 1)
 				)
@@
 		(in_pos_files yes)
 		(dnp no)
-		(property "Reference" "#PWR043"
+		(property "Reference" "#PWR061"
 			(at 194.31 74.93 0)
 			(hide yes)
@@
 			(project ""
 				(path "/bcc951e4-6780-442e-8e93-0576bc471757/f7e313ad-53b3-434b-b9a9-dc814318d635"
-					(reference "#PWR043")
+					(reference "#PWR061")
 					(unit 1)
 				)
@@
 		(in_pos_files yes)
 		(dnp no)
-		(property "Reference" "#PWR124"
+		(property "Reference" "#PWR048"
 			(at 95.25 72.39 0)
 			(hide yes)
@@
 			(project ""
 				(path "/bcc951e4-6780-442e-8e93-0576bc471757/f7e313ad-53b3-434b-b9a9-dc814318d635"
-					(reference "#PWR124")
+					(reference "#PWR048")
 					(unit 1)
 				)
@@
 		(in_pos_files yes)
 		(dnp no)
-		(property "Reference" "#PWR032"
+		(property "Reference" "#PWR049"
 			(at 101.6 53.34 0)
 			(hide yes)
@@
 				)
 				(path "/bcc951e4-6780-442e-8e93-0576bc471757/f7e313ad-53b3-434b-b9a9-dc814318d635"
-					(reference "#PWR032")
+					(reference "#PWR049")
 					(unit 1)
 				)
@@
 		(in_pos_files yes)
 		(dnp no)
-		(property "Reference" "#PWR035"
+		(property "Reference" "#PWR052"
 			(at 139.7 92.71 0)
 			(hide yes)
@@
 				)
 				(path "/bcc951e4-6780-442e-8e93-0576bc471757/f7e313ad-53b3-434b-b9a9-dc814318d635"
-					(reference "#PWR035")
+					(reference "#PWR052")
 					(unit 1)
 				)
@@
 		(in_pos_files yes)
 		(dnp no)
-		(property "Reference" "#PWR044"
+		(property "Reference" "#PWR062"
 			(at 200.66 114.3 0)
 			(hide yes)
@@
 			(project ""
 				(path "/bcc951e4-6780-442e-8e93-0576bc471757/f7e313ad-53b3-434b-b9a9-dc814318d635"
-					(reference "#PWR044")
+					(reference "#PWR062")
 					(unit 1)
 				)
@@
 		(in_pos_files yes)
 		(dnp no)
-		(property "Reference" "#PWR036"
+		(property "Reference" "#PWR053"
 			(at 148.59 86.36 0)
 			(hide yes)
@@
 				)
 				(path "/bcc951e4-6780-442e-8e93-0576bc471757/f7e313ad-53b3-434b-b9a9-dc814318d635"
-					(reference "#PWR036")
+					(reference "#PWR053")
 					(unit 1)
 				)
@@
 		(in_pos_files yes)
 		(dnp no)
-		(property "Reference" "#PWR0125"
+		(property "Reference" "#PWR055"
 			(at 149.86 91.44 0)
 			(hide yes)
@@
 			(project "fpv_drone"
 				(path "/bcc951e4-6780-442e-8e93-0576bc471757/f7e313ad-53b3-434b-b9a9-dc814318d635"
-					(reference "#PWR0125")
-					(unit 1)
-				)
+					(reference "#PWR055")
+					(unit 1)
+				)
