File: fpv_drone/peripherals.kicad_sch (KiCad schematic)
At the start: 6 parts, among them J1 BUZZER, J10 SWD_DEBUG, Q1 BSS138

Commit message: updated
Parts:
- J11: renamed from J1; footprint Connector_PinHeader_2.54mm:PinHeader_1x02_P2.54mm_Vertical -> Buzzer_Beeper:MagneticBuzzer_Kobitone_254-EMB84Q-RO
- J12: renamed from J10; footprint Connector_PinHeader_2.54mm:PinHeader_1x04_P2.54mm_Vertical -> Connector_PinHeader_1.27mm:PinHeader_1x04_P1.27mm_Vertical
- R15: renamed from R1; value 100k/100k -> 100k
- renumbered D1 to D3, Q1 to Q26, R12 to R16
Connections:
- net VBAT_SENSE: now also R15.2, R16.1; no longer R15.1
- new net +BATT: R15.1
Other:
- moved on the sheet: J12
