File: fpv_drone/power_supply.kicad_sch (KiCad schematic)
At the start: 22 parts, among them J2 BATT, U2 TPS54302_5V, U3 TPS54302_10V, U4 AMS1117-3.3

Commit message: updated
Parts:
- removed C10: 22µF, Capacitor_SMD:C_0805_2012Metric, symbol Device:C
- removed C5: 10µF, Capacitor_SMD:C_0805_2012Metric, symbol Device:C
- removed C6, C7: 100nF, Capacitor_SMD:C_0402_1005Metric, symbol Device:C
- removed L3: 4.7µH, Inductor_SMD:L_6.3x6.3_H3, symbol Device:L
- removed R4: 156k, Resistor_SMD:R_0402_1005Metric, symbol Device:R
- removed R5: 10k, Resistor_SMD:R_0402_1005Metric, symbol Device:R
- removed U3: TPS54302_10V, Package_TO_SOT_SMD:SOT-23-6, symbol Regulator_Switching:TPS54302
- C2: footprint Capacitor_SMD:CP_Elec_8x10.5 -> Capacitor_SMD:C_Elec_6.3x5.8
Connections:
- net GND: now also J2.1 (Pin_1); no longer J2.2 (Pin_2)
- net VBAT renamed +BATT
- net +BATT: now also J2.2 (Pin_2); no longer J2.1 (Pin_1)
Other:
- moved on the sheet: C3, C4, C8, C9, L2, R2, R3, U2
